File: Kicad/LED_DUAL_DRIVER.sch (KiCad schematic (older format))
At the start: 12 parts

Commit message: 
Connections:
- net GND: now also U?.8 (GND)
- net SRCLR_b: now reaches U?.10 (SRCLR_b)
- net SCLK: now reaches U?.11 (SRCLK)
- net LED_CS: now reaches U?.12 (RCLK)
- net OE_b: now reaches U?.13 (OE_b)
- net SDIN: now reaches U?.14 (SER)
- net SDOUT: now reaches U?.9 (QH')
Changed lines of the file:
@@
 LIBS:__xbee-pro
 LIBS:CAR
+LIBS:car_v3-cache
 EELAYER 27 0
 EELAYER END
@@
 Sheet 6 14
 Title ""
-Date "30 may 2014"
+Date "31 may 2014"
 Rev ""
 Comp ""
@@
 U 1 1 53880946
 P 3600 3200
+AR Path="/5387F9D3/53880946" Ref="U?"  Part="1"
+AR Path="/5387F99B/53880946" Ref="U?"  Part="1"
 F 0 "U?" H 3600 3750 60  0000 C CNN
 F 1 "SHFTREG_H" H 3600 2650 60  0000 C CNN
@@
 U 1 1 53880A57
 P 7150 2550
+AR Path="/5387F9D3/53880A57" Ref="J?"  Part="1"
+AR Path="/5387F99B/53880A57" Ref="J?"  Part="1"
 F 0 "J?" H 7150 2800 60  0000 C CNN
 F 1 "CONN_LED" H 7150 2300 60  0000 C CNN
@@
 U 1 1 53880A79
 P 6250 2450
+AR Path="/5387F9D3/53880A79" Ref="R?"  Part="1"
+AR Path="/5387F99B/53880A79" Ref="R?"  Part="1"
 F 0 "R?" V 6330 2450 40  0000 C CNN
 F 1 "R" V 6257 2451 40  0000 C CNN
@@
 U 1 1 53880A7F
 P 6250 2650
+AR Path="/5387F9D3/53880A7F" Ref="R?"  Part="1"
+AR Path="/5387F99B/53880A7F" Ref="R?"  Part="1"
 F 0 "R?" V 6330 2650 40  0000 C CNN
 F 1 "R" V 6257 2651 40  0000 C CNN
@@
 U 1 1 53880A85
 P 6250 2850
+AR Path="/5387F9D3/53880A85" Ref="R?"  Part="1"
+AR Path="/5387F99B/53880A85" Ref="R?"  Part="1"
 F 0 "R?" V 6330 2850 40  0000 C CNN
 F 1 "R" V 6257 2851 40  0000 C CNN
@@
 U 1 1 53880BE6
 P 7150 3450
+AR Path="/5387F9D3/53880BE6" Ref="J?"  Part="1"
+AR Path="/5387F99B/53880BE6" Ref="J?"  Part="1"
 F 0 "J?" H 7150 3700 60  0000 C CNN
 F 1 "CONN_LED" H 7150 3200 60  0000 C CNN
@@
 U 1 1 53880BEC
 P 6250 3350
+AR Path="/5387F9D3/53880BEC" Ref="R?"  Part="1"
+AR Path="/5387F99B/53880BEC" Ref="R?"  Part="1"
 F 0 "R?" V 6330 3350 40  0000 C CNN
 F 1 "R" V 6257 3351 40  0000 C CNN
@@
 U 1 1 53880BF2
 P 6250 3550
+AR Path="/5387F9D3/53880BF2" Ref="R?"  Part="1"
+AR Path="/5387F99B/53880BF2" Ref="R?"  Part="1"
 F 0 "R?" V 6330 3550 40  0000 C CNN
 F 1 "R" V 6257 3551 40  0000 C CNN
@@
 U 1 1 53880BF8
 P 6250 3750
+AR Path="/5387F9D3/53880BF8" Ref="R?"  Part="1"
+AR Path="/5387F99B/53880BF8" Ref="R?"  Part="1"
 F 0 "R?" V 6330 3750 40  0000 C CNN
 F 1 "R" V 6257 3751 40  0000 C CNN
@@
 U 1 1 53881290
 P 5300 3100
+AR Path="/5387F9D3/53881290" Ref="U?"  Part="1"
+AR Path="/5387F99B/53881290" Ref="U?"  Part="1"
 F 0 "U?" H 5300 3350 60  0000 C CNN
 F 1 "AO4828" H 5300 2850 60  0000 C CNN
@@
 U 1 1 538812D6
 P 5300 2500
+AR Path="/5387F9D3/538812D6" Ref="U?"  Part="1"
+AR Path="/5387F99B/538812D6" Ref="U?"  Part="1"
 F 0 "U?" H 5300 2750 60  0000 C CNN
 F 1 "AO4828" H 5300 2250 60  0000 C CNN
@@
 U 1 1 538812F1
 P 5300 3700
+AR Path="/5387F9D3/538812F1" Ref="U?"  Part="1"
+AR Path="/5387F99B/538812F1" Ref="U?"  Part="1"
 F 0 "U?" H 5300 3950 60  0000 C CNN
 F 1 "AO4828" H 5300 3450 60  0000 C CNN
@@
 	1    0    0    -1
 $EndComp
-Wire Wire Line
-	6650 2500 6500 2500
-Wire Wire Line
-	6500 2500 6500 2450
-Wire Wire Line
-	6650 2600 6500 2600
-Wire Wire Line
-	6500 2600 6500 2650
-Wire Wire Line
-	6650 2700 6650 2850
-Wire Wire Line
-	6650 2850 6500 2850
-Wire Wire Line
-	6650 2250 6650 2400
-Wire Wire Line
-	6250 2250 6650 2250
-Wire Wire Line
-	6650 3400 6500 3400
-Wire Wire Line
-	6500 3400 6500 3350
-Wire Wire Line
-	6650 3500 6500 3500
-Wire Wire Line
-	6500 3500 6500 3550
-Wire Wire Line
-	6650 3600 6650 3750
-Wire Wire Line
-	6650 3750 6500 3750
-Wire Wire Line
-	6650 3150 6650 3300
-Wire Wire Line
-	6250 3150 6650 3150
-Wire Wire Line
-	5800 2350 5800 2450
-Wire Wire Line
-	5800 2550 5800 2650
-Wire Wire Line
-	5800 2650 6000 2650
-Wire Wire Line
-	5800 2450 6000 2450
-Wire Wire Line
-	5800 2850 5800 3050
-Wire Wire Line
-	5800 2850 6000 2850
-Connection ~ 5800 2950
-Wire Wire Line
-	5800 3150 5800 3350
-Wire Wire Line
-	5800 3350 6000 3350
-Connection ~ 5800 3250
-Wire Wire Line
-	5800 3650 5800 3550
-Wire Wire Line
-	5800 3850 5800 3750
-Wire Wire Line
-	5800 3550 6000 3550
-Wire Wire Line
-	5800 3750 6000 3750
-Wire Wire Line
-	4800 2950 4700 2950
-Wire Wire Line
-	4700 3150 4800 3150
-Wire Wire Line
-	4700 3550 4800 3550
-Wire Wire Line
-	4700 3750 4800 3750
-Wire Wire Line
-	4800 2350 4700 2350
-Wire Wire Line
-	4700 2550 4800 2550
-Connection ~ 4700 2950
-Connection ~ 4700 3550
 $Comp
 L GND #PWR?
 U 1 1 53881504
 P 4700 3450
+AR Path="/5387F9D3/53881504" Ref="#PWR?"  Part="1"
+AR Path="/5387F99B/53881504" Ref="#PWR?"  Part="1"
 F 0 "#PWR?" H 4700 3450 30  0001 C CNN
 F 1 "GND" H 4700 3380 30  0001 C CNN
@@
 U 1 1 53881511
 P 4700 2850
+AR Path="/5387F9D3/53881511" Ref="#PWR?"  Part="1"
+AR Path="/5387F99B/53881511" Ref="#PWR?"  Part="1"
 F 0 "#PWR?" H 4700 2850 30  0001 C CNN
 F 1 "GND" H 4700 2780 30  0001 C CNN
@@
 U 1 1 53881517
 P 4700 2250
+AR Path="/5387F9D3/53881517" Ref="#PWR?"  Part="1"
+AR Path="/5387F99B/53881517" Ref="#PWR?"  Part="1"
 F 0 "#PWR?" H 4700 2250 30  0001 C CNN
 F 1 "GND" H 4700 2180 30  0001 C CNN
@@
 	-1   0    0    1
 $EndComp
-Wire Wire Line
-	4700 2250 4700 2550
-Connection ~ 4700 2350
-Wire Wire Line
-	4700 3450 4700 3750
-Wire Wire Line
-	4700 2850 4700 3150
-Wire Wire Line
-	4200 2450 4800 2450
-Wire Wire Line
-	4300 2650 4800 2650
-Wire Wire Line
-	4300 3850 4800 3850
-Wire Wire Line
-	4400 3650 4800 3650
-Wire Wire Line
-	4200 2450 4200 2850
-Wire Wire Line
-	4300 2650 4300 2950
-Wire Wire Line
-	4200 3050 4800 3050
-Wire Wire Line
-	4300 2950 4200 2950
-Wire Wire Line
-	4300 3850 4300 3350
-Wire Wire Line
-	4300 3350 4200 3350
-Wire Wire Line
-	4400 3650 4400 3250
-Wire Wire Line
-	4400 3250 4200 3250
-Wire Wire Line
-	4800 3250 4500 3250
-Wire Wire Line
-	4500 3250 4500 3150
-Wire Wire Line
-	4500 3150 4200 3150
 NoConn ~ 4200 3450
 NoConn ~ 4200 3550
@@
 U 1 1 53881AE0
 P 3000 2800
+AR Path="/5387F9D3/53881AE0" Ref="#PWR?"  Part="1"
+AR Path="/5387F99B/53881AE0" Ref="#PWR?"  Part="1"
 F 0 "#PWR?" H 3000 2760 30  0001 C CNN
 F 1 "+3.3V" H 3000 2910 30  0000 C CNN
@@
 	1    0    0    -1
 $EndComp
+Text GLabel 2600 3150 0    60   UnSpc ~ 0
+SCLK
+$Comp
+L GND #PWR?
+U 1 1 53897F20
+P 3000 3650
+F 0 "#PWR?" H 3000 3650 30  0001 C CNN
+F 1 "GND" H 3000 3580 30  0001 C CNN
+F 2 "" H 3000 3650 60  0000 C CNN
+F 3 "" H 3000 3650 60  0000 C CNN
+	1    3000 3650
+	1    0    0    -1
+$EndComp
+Text HLabel 3000 3050 0    60   UnSpc ~ 0
+SDOUT
+Text GLabel 3000 3450 0    60   UnSpc ~ 0
+OE_b
+Text HLabel 3000 2950 0    60   UnSpc ~ 0
+SDIN
+Text GLabel 2600 3350 0    60   UnSpc ~ 0
+SRCLR_b
+Wire Wire Line
+	6650 2500 6500 2500
+Wire Wire Line
+	6500 2500 6500 2450
+Wire Wire Line
+	6650 2600 6500 2600
+Wire Wire Line
+	6500 2600 6500 2650
+Wire Wire Line
+	6650 2700 6650 2850
+Wire Wire Line
+	6650 2850 6500 2850
+Wire Wire Line
+	6650 2250 6650 2400
+Wire Wire Line
+	6250 2250 6650 2250
+Wire Wire Line
+	6650 3400 6500 3400
+Wire Wire Line
+	6500 3400 6500 3350
+Wire Wire Line
+	6650 3500 6500 3500
+Wire Wire Line
+	6500 3500 6500 3550
+Wire Wire Line
+	6650 3600 6650 3750
+Wire Wire Line
+	6650 3750 6500 3750
+Wire Wire Line
+	6650 3150 6650 3300
+Wire Wire Line
+	6250 3150 6650 3150
+Wire Wire Line
+	5800 2350 5800 2450
+Wire Wire Line
+	5800 2550 5800 2650
+Wire Wire Line
+	5800 2650 6000 2650
+Wire Wire Line
+	5800 2450 6000 2450
+Wire Wire Line
+	5800 2850 5800 2950
+Wire Wire Line
+	5800 2950 5800 3050
+Wire Wire Line
+	5800 2850 6000 2850
+Connection ~ 5800 2950
+Wire Wire Line
+	5800 3150 5800 3250
+Wire Wire Line
+	5800 3250 5800 3350
+Wire Wire Line
+	5800 3350 6000 3350
+Connection ~ 5800 3250
+Wire Wire Line
+	5800 3650 5800 3550
+Wire Wire Line
+	5800 3850 5800 3750
+Wire Wire Line
+	5800 3550 6000 3550
+Wire Wire Line
+	5800 3750 6000 3750
+Wire Wire Line
+	4800 2950 4700 2950
+Wire Wire Line
+	4700 3150 4800 3150
+Wire Wire Line
+	4700 3550 4800 3550
+Wire Wire Line
+	4700 3750 4800 3750
+Wire Wire Line
+	4800 2350 4700 2350
+Wire Wire Line
+	4700 2550 4800 2550
+Connection ~ 4700 2950
+Connection ~ 4700 3550
+Wire Wire Line
+	4700 2250 4700 2350
+Wire Wire Line
+	4700 2350 4700 2550
+Connection ~ 4700 2350
+Wire Wire Line
+	4700 3450 4700 3550
+Wire Wire Line
+	4700 3550 4700 3750
+Wire Wire Line
+	4700 2850 4700 2950
+Wire Wire Line
+	4700 2950 4700 3150
+Wire Wire Line
+	4200 2450 4800 2450
+Wire Wire Line
+	4300 2650 4800 2650
+Wire Wire Line
+	4300 3850 4800 3850
+Wire Wire Line
+	4400 3650 4800 3650
+Wire Wire Line
+	4200 2450 4200 2850
+Wire Wire Line
+	4300 2650 4300 2950
+Wire Wire Line
+	4200 3050 4800 3050
+Wire Wire Line
+	4300 2950 4200 2950
+Wire Wire Line
+	4300 3850 4300 3350
+Wire Wire Line
+	4300 3350 4200 3350
+Wire Wire Line
+	4400 3650 4400 3250
+Wire Wire Line
+	4400 3250 4200 3250
+Wire Wire Line
+	4800 3250 4500 3250
+Wire Wire Line
+	4500 3250 4500 3150
+Wire Wire Line
+	4500 3150 4200 3150
 Wire Wire Line
 	3000 2800 3000 2850
+Wire Wire Line
+	3000 3550 3000 3650
+Wire Wire Line
+	3000 3150 2600 3150
+Wire Wire Line
+	2600 3350 3000 3350
+Text GLabel 3000 3250 0    60   UnSpc ~ 0
+LED_CS
 $EndSCHEMATC

Commit message: 
Connections:
- net SDIN renamed LED_SDIN
- net SDOUT renamed LED_SDOUT
Changed lines of the file:
@@
 Sheet 6 14
 Title ""
-Date "31 may 2014"
+Date "1 jun 2014"
 Rev ""
 Comp ""
@@
 $EndComp
 Text HLabel 3000 3050 0    60   UnSpc ~ 0
-SDOUT
+LED_SDOUT
 Text GLabel 3000 3450 0    60   UnSpc ~ 0
 OE_b
 Text HLabel 3000 2950 0    60   UnSpc ~ 0
-SDIN
+LED_SDIN
 Text GLabel 2600 3350 0    60   UnSpc ~ 0
 SRCLR_b

Commit message: 
Parts:
- gave numbers to parts that had none: 12
Changed lines of the file:
@@
 $Descr A4 11693 8268
 encoding utf-8
-Sheet 6 14
+Sheet 7 15
 Title ""
 Date "1 jun 2014"
@@
 $EndDescr
 $Comp
-L SHFTREG_H U?
+L SHFTREG_H U9
 U 1 1 53880946
 P 3600 3200
-AR Path="/5387F9D3/53880946" Ref="U?"  Part="1"
-AR Path="/5387F99B/53880946" Ref="U?"  Part="1"
-F 0 "U?" H 3600 3750 60  0000 C CNN
+AR Path="/5387F99B/53880946" Ref="U9"  Part="1"
+AR Path="/5387F9D3/53880946" Ref="U13"  Part="1"
+F 0 "U13" H 3600 3750 60  0000 C CNN
 F 1 "SHFTREG_H" H 3600 2650 60  0000 C CNN
 F 2 "~" V 3350 3300 60  0000 C CNN
@@
 $EndComp
 $Comp
-L CONN_LED J?
+L CONN_LED J5
 U 1 1 53880A57
 P 7150 2550
-AR Path="/5387F9D3/53880A57" Ref="J?"  Part="1"
-AR Path="/5387F99B/53880A57" Ref="J?"  Part="1"
-F 0 "J?" H 7150 2800 60  0000 C CNN
+AR Path="/5387F99B/53880A57" Ref="J5"  Part="1"
+AR Path="/5387F9D3/53880A57" Ref="J7"  Part="1"
+F 0 "J7" H 7150 2800 60  0000 C CNN
 F 1 "CONN_LED" H 7150 2300 60  0000 C CNN
 F 2 "~" H 7000 2500 60  0000 C CNN
@@
 $EndComp
 $Comp
-L R R?
+L R R9
 U 1 1 53880A79
 P 6250 2450
-AR Path="/5387F9D3/53880A79" Ref="R?"  Part="1"
-AR Path="/5387F99B/53880A79" Ref="R?"  Part="1"
-F 0 "R?" V 6330 2450 40  0000 C CNN
+AR Path="/5387F99B/53880A79" Ref="R9"  Part="1"
+AR Path="/5387F9D3/53880A79" Ref="R15"  Part="1"
+F 0 "R15" V 6330 2450 40  0000 C CNN
 F 1 "R" V 6257 2451 40  0000 C CNN
 F 2 "~" V 6180 2450 30  0000 C CNN
@@
 $EndComp
 $Comp
-L R R?
+L R R10
 U 1 1 53880A7F
 P 6250 2650
-AR Path="/5387F9D3/53880A7F" Ref="R?"  Part="1"
-AR Path="/5387F99B/53880A7F" Ref="R?"  Part="1"
-F 0 "R?" V 6330 2650 40  0000 C CNN
+AR Path="/5387F99B/53880A7F" Ref="R10"  Part="1"
+AR Path="/5387F9D3/53880A7F" Ref="R16"  Part="1"
+F 0 "R16" V 6330 2650 40  0000 C CNN
 F 1 "R" V 6257 2651 40  0000 C CNN
 F 2 "~" V 6180 2650 30  0000 C CNN
@@
 $EndComp
 $Comp
-L R R?
+L R R11
 U 1 1 53880A85
 P 6250 2850
-AR Path="/5387F9D3/53880A85" Ref="R?"  Part="1"
-AR Path="/5387F99B/53880A85" Ref="R?"  Part="1"
-F 0 "R?" V 6330 2850 40  0000 C CNN
+AR Path="/5387F99B/53880A85" Ref="R11"  Part="1"
+AR Path="/5387F9D3/53880A85" Ref="R17"  Part="1"
+F 0 "R17" V 6330 2850 40  0000 C CNN
 F 1 "R" V 6257 2851 40  0000 C CNN
 F 2 "~" V 6180 2850 30  0000 C CNN
@@
 8V
 $Comp
-L CONN_LED J?
+L CONN_LED J6
 U 1 1 53880BE6
 P 7150 3450
-AR Path="/5387F9D3/53880BE6" Ref="J?"  Part="1"
-AR Path="/5387F99B/53880BE6" Ref="J?"  Part="1"
-F 0 "J?" H 7150 3700 60  0000 C CNN
+AR Path="/5387F99B/53880BE6" Ref="J6"  Part="1"
+AR Path="/5387F9D3/53880BE6" Ref="J8"  Part="1"
+F 0 "J8" H 7150 3700 60  0000 C CNN
 F 1 "CONN_LED" H 7150 3200 60  0000 C CNN
 F 2 "~" H 7000 3400 60  0000 C CNN
@@
 $EndComp
 $Comp
-L R R?
+L R R12
 U 1 1 53880BEC
 P 6250 3350
-AR Path="/5387F9D3/53880BEC" Ref="R?"  Part="1"
-AR Path="/5387F99B/53880BEC" Ref="R?"  Part="1"
-F 0 "R?" V 6330 3350 40  0000 C CNN
+AR Path="/5387F99B/53880BEC" Ref="R12"  Part="1"
+AR Path="/5387F9D3/53880BEC" Ref="R18"  Part="1"
+F 0 "R18" V 6330 3350 40  0000 C CNN
 F 1 "R" V 6257 3351 40  0000 C CNN
 F 2 "~" V 6180 3350 30  0000 C CNN
@@
 $EndComp
 $Comp
-L R R?
+L R R13
 U 1 1 53880BF2
 P 6250 3550
-AR Path="/5387F9D3/53880BF2" Ref="R?"  Part="1"
-AR Path="/5387F99B/53880BF2" Ref="R?"  Part="1"
-F 0 "R?" V 6330 3550 40  0000 C CNN
+AR Path="/5387F99B/53880BF2" Ref="R13"  Part="1"
+AR Path="/5387F9D3/53880BF2" Ref="R19"  Part="1"
+F 0 "R19" V 6330 3550 40  0000 C CNN
 F 1 "R" V 6257 3551 40  0000 C CNN
 F 2 "~" V 6180 3550 30  0000 C CNN
@@
 $EndComp
 $Comp
-L R R?
+L R R14
 U 1 1 53880BF8
 P 6250 3750
-AR Path="/5387F9D3/53880BF8" Ref="R?"  Part="1"
-AR Path="/5387F99B/53880BF8" Ref="R?"  Part="1"
-F 0 "R?" V 6330 3750 40  0000 C CNN
+AR Path="/5387F99B/53880BF8" Ref="R14"  Part="1"
+AR Path="/5387F9D3/53880BF8" Ref="R20"  Part="1"
+F 0 "R20" V 6330 3750 40  0000 C CNN
 F 1 "R" V 6257 3751 40  0000 C CNN
 F 2 "~" V 6180 3750 30  0000 C CNN
@@
 8V
 $Comp
-L AO4828 U?
+L AO4828 U11
 U 1 1 53881290
 P 5300 3100
-AR Path="/5387F9D3/53881290" Ref="U?"  Part="1"
-AR Path="/5387F99B/53881290" Ref="U?"  Part="1"
-F 0 "U?" H 5300 3350 60  0000 C CNN
+AR Path="/5387F99B/53881290" Ref="U11"  Part="1"
+AR Path="/5387F9D3/53881290" Ref="U15"  Part="1"
+F 0 "U15" H 5300 3350 60  0000 C CNN
 F 1 "AO4828" H 5300 2850 60  0000 C CNN
 F 2 "~" H 5250 2650 60  0000 C CNN
@@
 $EndComp
 $Comp
-L AO4828 U?
+L AO4828 U10
 U 1 1 538812D6
 P 5300 2500
-AR Path="/5387F9D3/538812D6" Ref="U?"  Part="1"
-AR Path="/5387F99B/538812D6" Ref="U?"  Part="1"
-F 0 "U?" H 5300 2750 60  0000 C CNN
+AR Path="/5387F99B/538812D6" Ref="U10"  Part="1"
+AR Path="/5387F9D3/538812D6" Ref="U14"  Part="1"
+F 0 "U14" H 5300 2750 60  0000 C CNN
 F 1 "AO4828" H 5300 2250 60  0000 C CNN
 F 2 "~" H 5250 2050 60  0000 C CNN
@@
 $EndComp
 $Comp
-L AO4828 U?
+L AO4828 U12
 U 1 1 538812F1
 P 5300 3700
-AR Path="/5387F9D3/538812F1" Ref="U?"  Part="1"
-AR Path="/5387F99B/538812F1" Ref="U?"  Part="1"
-F 0 "U?" H 5300 3950 60  0000 C CNN
+AR Path="/5387F99B/538812F1" Ref="U12"  Part="1"
+AR Path="/5387F9D3/538812F1" Ref="U16"  Part="1"
+F 0 "U16" H 5300 3950 60  0000 C CNN
 F 1 "AO4828" H 5300 3450 60  0000 C CNN
 F 2 "~" H 5250 3250 60  0000 C CNN
@@
 $EndComp
 $Comp
-L GND #PWR?
+L GND #PWR041
 U 1 1 53881504
 P 4700 3450
-AR Path="/5387F9D3/53881504" Ref="#PWR?"  Part="1"
-AR Path="/5387F99B/53881504" Ref="#PWR?"  Part="1"
-F 0 "#PWR?" H 4700 3450 30  0001 C CNN
+AR Path="/5387F99B/53881504" Ref="#PWR041"  Part="1"
+AR Path="/5387F9D3/53881504" Ref="#PWR046"  Part="1"
+F 0 "#PWR046" H 4700 3450 30  0001 C CNN
 F 1 "GND" H 4700 3380 30  0001 C CNN
 F 2 "" H 4700 3450 60  0000 C CNN
@@
 $EndComp
 $Comp
-L GND #PWR?
+L GND #PWR042
 U 1 1 53881511
 P 4700 2850
-AR Path="/5387F9D3/53881511" Ref="#PWR?"  Part="1"
-AR Path="/5387F99B/53881511" Ref="#PWR?"  Part="1"
-F 0 "#PWR?" H 4700 2850 30  0001 C CNN
+AR Path="/5387F99B/53881511" Ref="#PWR042"  Part="1"
+AR Path="/5387F9D3/53881511" Ref="#PWR047"  Part="1"
+F 0 "#PWR047" H 4700 2850 30  0001 C CNN
 F 1 "GND" H 4700 2780 30  0001 C CNN
 F 2 "" H 4700 2850 60  0000 C CNN
@@
 $EndComp
 $Comp
-L GND #PWR?
+L GND #PWR043
 U 1 1 53881517
 P 4700 2250
-AR Path="/5387F9D3/53881517" Ref="#PWR?"  Part="1"
-AR Path="/5387F99B/53881517" Ref="#PWR?"  Part="1"
-F 0 "#PWR?" H 4700 2250 30  0001 C CNN
+AR Path="/5387F99B/53881517" Ref="#PWR043"  Part="1"
+AR Path="/5387F9D3/53881517" Ref="#PWR048"  Part="1"
+F 0 "#PWR048" H 4700 2250 30  0001 C CNN
 F 1 "GND" H 4700 2180 30  0001 C CNN
 F 2 "" H 4700 2250 60  0000 C CNN
@@
 NoConn ~ 4200 3550
 $Comp
-L +3.3V #PWR?
+L +3.3V #PWR044
 U 1 1 53881AE0
 P 3000 2800
-AR Path="/5387F9D3/53881AE0" Ref="#PWR?"  Part="1"
-AR Path="/5387F99B/53881AE0" Ref="#PWR?"  Part="1"
-F 0 "#PWR?" H 3000 2760 30  0001 C CNN
+AR Path="/5387F99B/53881AE0" Ref="#PWR044"  Part="1"
+AR Path="/5387F9D3/53881AE0" Ref="#PWR049"  Part="1"
+F 0 "#PWR049" H 3000 2760 30  0001 C CNN
 F 1 "+3.3V" H 3000 2910 30  0000 C CNN
 F 2 "" H 3000 2800 60  0000 C CNN
@@
 SCLK
 $Comp
-L GND #PWR?
+L GND #PWR045
 U 1 1 53897F20
 P 3000 3650
-F 0 "#PWR?" H 3000 3650 30  0001 C CNN
+AR Path="/5387F99B/53897F20" Ref="#PWR045"  Part="1"
+AR Path="/5387F9D3/53897F20" Ref="#PWR050"  Part="1"
+F 0 "#PWR050" H 3000 3650 30  0001 C CNN
 F 1 "GND" H 3000 3580 30  0001 C CNN
 F 2 "" H 3000 3650 60  0000 C CNN
@@
 	5800 2450 6000 2450
 Wire Wire Line
-	5800 2850 5800 2950
-Wire Wire Line
-	5800 2950 5800 3050
+	5800 2850 5800 3050
 Wire Wire Line
 	5800 2850 6000 2850
 Connection ~ 5800 2950
 Wire Wire Line
-	5800 3150 5800 3250
-Wire Wire Line
-	5800 3250 5800 3350
+	5800 3150 5800 3350
 Wire Wire Line
 	5800 3350 6000 3350
@@
 Connection ~ 4700 3550
 Wire Wire Line
-	4700 2250 4700 2350
-Wire Wire Line
-	4700 2350 4700 2550
+	4700 2250 4700 2550
 Connection ~ 4700 2350
 Wire Wire Line
-	4700 3450 4700 3550
-Wire Wire Line
-	4700 3550 4700 3750
-Wire Wire Line
-	4700 2850 4700 2950
-Wire Wire Line
-	4700 2950 4700 3150
+	4700 3450 4700 3750
+Wire Wire Line
+	4700 2850 4700 3150
 Wire Wire Line
 	4200 2450 4800 2450
