File: Kicad/LED_DUAL_DRIVER.sch (KiCad schematic (older format))
At the start: 12 parts, among them J5 CONN_LED, J6 CONN_LED, U10 AO4828, U11 AO4828, U12 AO4828, U9 SHFTREG_H

Commit message: 
Parts:
- renumbered J5 to J2, J6 to J3, R9 to R3, R10 to R4, R11 to R5, R12 to R6, R13 to R7, R14 to R8, U9 to U3, U10 to U4, U11 to U5, U12 to U6
Connections:
- net LED_CS renamed CS
Changed lines of the file:
@@
 $Descr A4 11693 8268
 encoding utf-8
-Sheet 6 15
+Sheet 4 15
 Title ""
-Date "1 jun 2014"
+Date "7 jun 2014"
 Rev ""
 Comp ""
@@
 $EndDescr
 $Comp
-L SHFTREG_H U9
+L SHFTREG_H U3
 U 1 1 53880946
 P 3600 3200
-AR Path="/5387F99B/53880946" Ref="U9"  Part="1"
-AR Path="/5387F9D3/53880946" Ref="U13"  Part="1"
-F 0 "U9" H 3600 3750 60  0000 C CNN
+AR Path="/5387F99B/53880946" Ref="U3"  Part="1"
+AR Path="/5387F9D3/53880946" Ref="U7"  Part="1"
+F 0 "U7" H 3600 3750 60  0000 C CNN
 F 1 "SHFTREG_H" H 3600 2650 60  0000 C CNN
 F 2 "~" V 3350 3300 60  0000 C CNN
@@
 $EndComp
 $Comp
-L CONN_LED J5
+L CONN_LED J2
 U 1 1 53880A57
 P 7150 2550
-AR Path="/5387F99B/53880A57" Ref="J5"  Part="1"
-AR Path="/5387F9D3/53880A57" Ref="J7"  Part="1"
-F 0 "J5" H 7150 2800 60  0000 C CNN
+AR Path="/5387F99B/53880A57" Ref="J2"  Part="1"
+AR Path="/5387F9D3/53880A57" Ref="J4"  Part="1"
+F 0 "J4" H 7150 2800 60  0000 C CNN
 F 1 "CONN_LED" H 7150 2300 60  0000 C CNN
 F 2 "~" H 7000 2500 60  0000 C CNN
@@
 $EndComp
 $Comp
-L R R9
+L R R3
 U 1 1 53880A79
 P 6250 2450
-AR Path="/5387F99B/53880A79" Ref="R9"  Part="1"
-AR Path="/5387F9D3/53880A79" Ref="R15"  Part="1"
+AR Path="/5387F99B/53880A79" Ref="R3"  Part="1"
+AR Path="/5387F9D3/53880A79" Ref="R9"  Part="1"
 F 0 "R9" V 6330 2450 40  0000 C CNN
 F 1 "R" V 6257 2451 40  0000 C CNN
@@
 $EndComp
 $Comp
-L R R10
+L R R4
 U 1 1 53880A7F
 P 6250 2650
-AR Path="/5387F99B/53880A7F" Ref="R10"  Part="1"
-AR Path="/5387F9D3/53880A7F" Ref="R16"  Part="1"
+AR Path="/5387F99B/53880A7F" Ref="R4"  Part="1"
+AR Path="/5387F9D3/53880A7F" Ref="R10"  Part="1"
 F 0 "R10" V 6330 2650 40  0000 C CNN
 F 1 "R" V 6257 2651 40  0000 C CNN
@@
 $EndComp
 $Comp
-L R R11
+L R R5
 U 1 1 53880A85
 P 6250 2850
-AR Path="/5387F99B/53880A85" Ref="R11"  Part="1"
-AR Path="/5387F9D3/53880A85" Ref="R17"  Part="1"
+AR Path="/5387F99B/53880A85" Ref="R5"  Part="1"
+AR Path="/5387F9D3/53880A85" Ref="R11"  Part="1"
 F 0 "R11" V 6330 2850 40  0000 C CNN
 F 1 "R" V 6257 2851 40  0000 C CNN
@@
 $EndComp
 $Comp
-L CONN_LED J6
+L CONN_LED J3
 U 1 1 53880BE6
 P 7150 3450
-AR Path="/5387F99B/53880BE6" Ref="J6"  Part="1"
-AR Path="/5387F9D3/53880BE6" Ref="J8"  Part="1"
-F 0 "J6" H 7150 3700 60  0000 C CNN
+AR Path="/5387F99B/53880BE6" Ref="J3"  Part="1"
+AR Path="/5387F9D3/53880BE6" Ref="J5"  Part="1"
+F 0 "J5" H 7150 3700 60  0000 C CNN
 F 1 "CONN_LED" H 7150 3200 60  0000 C CNN
 F 2 "~" H 7000 3400 60  0000 C CNN
@@
 $EndComp
 $Comp
-L R R12
+L R R6
 U 1 1 53880BEC
 P 6250 3350
-AR Path="/5387F99B/53880BEC" Ref="R12"  Part="1"
-AR Path="/5387F9D3/53880BEC" Ref="R18"  Part="1"
+AR Path="/5387F99B/53880BEC" Ref="R6"  Part="1"
+AR Path="/5387F9D3/53880BEC" Ref="R12"  Part="1"
 F 0 "R12" V 6330 3350 40  0000 C CNN
 F 1 "R" V 6257 3351 40  0000 C CNN
@@
 $EndComp
 $Comp
-L R R13
+L R R7
 U 1 1 53880BF2
 P 6250 3550
-AR Path="/5387F99B/53880BF2" Ref="R13"  Part="1"
-AR Path="/5387F9D3/53880BF2" Ref="R19"  Part="1"
+AR Path="/5387F99B/53880BF2" Ref="R7"  Part="1"
+AR Path="/5387F9D3/53880BF2" Ref="R13"  Part="1"
 F 0 "R13" V 6330 3550 40  0000 C CNN
 F 1 "R" V 6257 3551 40  0000 C CNN
@@
 $EndComp
 $Comp
-L R R14
+L R R8
 U 1 1 53880BF8
 P 6250 3750
-AR Path="/5387F99B/53880BF8" Ref="R14"  Part="1"
-AR Path="/5387F9D3/53880BF8" Ref="R20"  Part="1"
+AR Path="/5387F99B/53880BF8" Ref="R8"  Part="1"
+AR Path="/5387F9D3/53880BF8" Ref="R14"  Part="1"
 F 0 "R14" V 6330 3750 40  0000 C CNN
 F 1 "R" V 6257 3751 40  0000 C CNN
@@
 $EndComp
 $Comp
-L AO4828 U11
+L AO4828 U5
 U 1 1 53881290
 P 5300 3100
-AR Path="/5387F99B/53881290" Ref="U11"  Part="1"
-AR Path="/5387F9D3/53881290" Ref="U15"  Part="1"
-F 0 "U11" H 5300 3350 60  0000 C CNN
+AR Path="/5387F99B/53881290" Ref="U5"  Part="1"
+AR Path="/5387F9D3/53881290" Ref="U9"  Part="1"
+F 0 "U9" H 5300 3350 60  0000 C CNN
 F 1 "AO4828" H 5300 2850 60  0000 C CNN
 F 2 "~" H 5250 2650 60  0000 C CNN
@@
 $EndComp
 $Comp
-L AO4828 U10
+L AO4828 U4
 U 1 1 538812D6
 P 5300 2500
-AR Path="/5387F99B/538812D6" Ref="U10"  Part="1"
-AR Path="/5387F9D3/538812D6" Ref="U14"  Part="1"
-F 0 "U10" H 5300 2750 60  0000 C CNN
+AR Path="/5387F99B/538812D6" Ref="U4"  Part="1"
+AR Path="/5387F9D3/538812D6" Ref="U8"  Part="1"
+F 0 "U8" H 5300 2750 60  0000 C CNN
 F 1 "AO4828" H 5300 2250 60  0000 C CNN
 F 2 "~" H 5250 2050 60  0000 C CNN
@@
 $EndComp
 $Comp
-L AO4828 U12
+L AO4828 U6
 U 1 1 538812F1
 P 5300 3700
-AR Path="/5387F99B/538812F1" Ref="U12"  Part="1"
-AR Path="/5387F9D3/538812F1" Ref="U16"  Part="1"
-F 0 "U12" H 5300 3950 60  0000 C CNN
+AR Path="/5387F99B/538812F1" Ref="U6"  Part="1"
+AR Path="/5387F9D3/538812F1" Ref="U10"  Part="1"
+F 0 "U10" H 5300 3950 60  0000 C CNN
 F 1 "AO4828" H 5300 3450 60  0000 C CNN
 F 2 "~" H 5250 3250 60  0000 C CNN
@@
 $EndComp
 $Comp
-L GND #PWR041
+L GND #PWR016
 U 1 1 53881504
 P 4700 3450
-AR Path="/5387F99B/53881504" Ref="#PWR041"  Part="1"
-AR Path="/5387F9D3/53881504" Ref="#PWR048"  Part="1"
-F 0 "#PWR048" H 4700 3450 30  0001 C CNN
+AR Path="/5387F99B/53881504" Ref="#PWR016"  Part="1"
+AR Path="/5387F9D3/53881504" Ref="#PWR023"  Part="1"
+F 0 "#PWR023" H 4700 3450 30  0001 C CNN
 F 1 "GND" H 4700 3380 30  0001 C CNN
 F 2 "" H 4700 3450 60  0000 C CNN
@@
 $EndComp
 $Comp
-L GND #PWR042
+L GND #PWR017
 U 1 1 53881511
 P 4700 2850
-AR Path="/5387F99B/53881511" Ref="#PWR042"  Part="1"
-AR Path="/5387F9D3/53881511" Ref="#PWR049"  Part="1"
-F 0 "#PWR049" H 4700 2850 30  0001 C CNN
+AR Path="/5387F99B/53881511" Ref="#PWR017"  Part="1"
+AR Path="/5387F9D3/53881511" Ref="#PWR024"  Part="1"
+F 0 "#PWR024" H 4700 2850 30  0001 C CNN
 F 1 "GND" H 4700 2780 30  0001 C CNN
 F 2 "" H 4700 2850 60  0000 C CNN
@@
 $EndComp
 $Comp
-L GND #PWR043
+L GND #PWR018
 U 1 1 53881517
 P 4700 2250
-AR Path="/5387F99B/53881517" Ref="#PWR043"  Part="1"
-AR Path="/5387F9D3/53881517" Ref="#PWR050"  Part="1"
-F 0 "#PWR050" H 4700 2250 30  0001 C CNN
+AR Path="/5387F99B/53881517" Ref="#PWR018"  Part="1"
+AR Path="/5387F9D3/53881517" Ref="#PWR025"  Part="1"
+F 0 "#PWR025" H 4700 2250 30  0001 C CNN
 F 1 "GND" H 4700 2180 30  0001 C CNN
 F 2 "" H 4700 2250 60  0000 C CNN
@@
 NoConn ~ 4200 3550
 $Comp
-L +3.3V #PWR044
+L +3.3V #PWR019
 U 1 1 53881AE0
 P 3000 2800
-AR Path="/5387F99B/53881AE0" Ref="#PWR044"  Part="1"
-AR Path="/5387F9D3/53881AE0" Ref="#PWR051"  Part="1"
-F 0 "#PWR051" H 3000 2760 30  0001 C CNN
+AR Path="/5387F99B/53881AE0" Ref="#PWR019"  Part="1"
+AR Path="/5387F9D3/53881AE0" Ref="#PWR026"  Part="1"
+F 0 "#PWR026" H 3000 2760 30  0001 C CNN
 F 1 "+3.3V" H 3000 2910 30  0000 C CNN
 F 2 "" H 3000 2800 60  0000 C CNN
@@
 	1    0    0    -1
 $EndComp
-Text GLabel 2600 3150 0    60   UnSpc ~ 0
-SCLK
-$Comp
-L GND #PWR045
+$Comp
+L GND #PWR020
 U 1 1 53897F20
 P 3000 3650
-AR Path="/5387F99B/53897F20" Ref="#PWR045"  Part="1"
-AR Path="/5387F9D3/53897F20" Ref="#PWR052"  Part="1"
-F 0 "#PWR052" H 3000 3650 30  0001 C CNN
+AR Path="/5387F99B/53897F20" Ref="#PWR020"  Part="1"
+AR Path="/5387F9D3/53897F20" Ref="#PWR027"  Part="1"
+F 0 "#PWR027" H 3000 3650 30  0001 C CNN
 F 1 "GND" H 3000 3580 30  0001 C CNN
 F 2 "" H 3000 3650 60  0000 C CNN
@@
 Text HLabel 3000 3050 0    60   UnSpc ~ 0
 LED_SDOUT
-Text GLabel 3000 3450 0    60   UnSpc ~ 0
-OE_b
 Text HLabel 3000 2950 0    60   UnSpc ~ 0
 LED_SDIN
-Text GLabel 2600 3350 0    60   UnSpc ~ 0
-SRCLR_b
 Wire Wire Line
 	6650 2500 6500 2500
@@
 Wire Wire Line
 	2600 3350 3000 3350
-Text GLabel 3000 3250 0    60   UnSpc ~ 0
-LED_CS
-$Comp
-L +8V #PWR046
-U 1 1 538B7840
+$Comp
+L +8V #PWR021
+U 1 1 538B7495
 P 6250 2250
-AR Path="/5387F99B/538B7840" Ref="#PWR046"  Part="1"
-AR Path="/5387F9D3/538B7840" Ref="#PWR053"  Part="1"
-F 0 "#PWR053" H 6250 2220 20  0001 C CNN
+AR Path="/5387F99B/538B7495" Ref="#PWR021"  Part="1"
+AR Path="/5387F9D3/538B7495" Ref="#PWR028"  Part="1"
+F 0 "#PWR028" H 6250 2220 20  0001 C CNN
 F 1 "+8V" H 6250 2360 30  0000 C CNN
 F 2 "" H 6250 2250 60  0000 C CNN
@@
 $EndComp
 $Comp
-L +8V #PWR047
-U 1 1 538B784D
+L +8V #PWR022
+U 1 1 538B74AC
 P 6250 3150
-AR Path="/5387F99B/538B784D" Ref="#PWR047"  Part="1"
-AR Path="/5387F9D3/538B784D" Ref="#PWR054"  Part="1"
-F 0 "#PWR054" H 6250 3120 20  0001 C CNN
+AR Path="/5387F99B/538B74AC" Ref="#PWR022"  Part="1"
+AR Path="/5387F9D3/538B74AC" Ref="#PWR029"  Part="1"
+F 0 "#PWR029" H 6250 3120 20  0001 C CNN
 F 1 "+8V" H 6250 3260 30  0000 C CNN
 F 2 "" H 6250 3150 60  0000 C CNN
@@
 	1    0    0    -1
 $EndComp
+Text HLabel 2600 3150 0    60   UnSpc ~ 0
+SCLK
+Text HLabel 3000 3250 0    60   UnSpc ~ 0
+CS
+Text HLabel 2600 3350 0    60   UnSpc ~ 0
+SRCLR_b
+Text HLabel 3000 3450 0    60   UnSpc ~ 0
+OE_b
 $EndSCHEMATC

Commit message: All wired. ERC passes with no errors. Might be good to go.
Connections:
- net LED_SDIN renamed SDIN
- net LED_SDOUT renamed SDOUT
Changed lines of the file:
@@
 $Descr A4 11693 8268
 encoding utf-8
-Sheet 4 15
+Sheet 3 15
 Title ""
-Date "7 jun 2014"
+Date "8 jun 2014"
 Rev ""
 Comp ""
@@
 U 1 1 53880946
 P 3600 3200
-AR Path="/5387F99B/53880946" Ref="U3"  Part="1"
-AR Path="/5387F9D3/53880946" Ref="U7"  Part="1"
-F 0 "U7" H 3600 3750 60  0000 C CNN
+AR Path="/5387F9D3/53880946" Ref="U3"  Part="1"
+AR Path="/539441D7/53880946" Ref="U13"  Part="1"
+F 0 "U3" H 3600 3750 60  0000 C CNN
 F 1 "SHFTREG_H" H 3600 2650 60  0000 C CNN
 F 2 "~" V 3350 3300 60  0000 C CNN
@@
 U 1 1 53880A57
 P 7150 2550
-AR Path="/5387F99B/53880A57" Ref="J2"  Part="1"
-AR Path="/5387F9D3/53880A57" Ref="J4"  Part="1"
-F 0 "J4" H 7150 2800 60  0000 C CNN
+AR Path="/5387F9D3/53880A57" Ref="J2"  Part="1"
+AR Path="/539441D7/53880A57" Ref="J15"  Part="1"
+F 0 "J2" H 7150 2800 60  0000 C CNN
 F 1 "CONN_LED" H 7150 2300 60  0000 C CNN
 F 2 "~" H 7000 2500 60  0000 C CNN
@@
 U 1 1 53880A79
 P 6250 2450
-AR Path="/5387F99B/53880A79" Ref="R3"  Part="1"
-AR Path="/5387F9D3/53880A79" Ref="R9"  Part="1"
-F 0 "R9" V 6330 2450 40  0000 C CNN
+AR Path="/5387F9D3/53880A79" Ref="R3"  Part="1"
+AR Path="/539441D7/53880A79" Ref="R15"  Part="1"
+F 0 "R3" V 6330 2450 40  0000 C CNN
 F 1 "R" V 6257 2451 40  0000 C CNN
 F 2 "~" V 6180 2450 30  0000 C CNN
@@
 U 1 1 53880A7F
 P 6250 2650
-AR Path="/5387F99B/53880A7F" Ref="R4"  Part="1"
-AR Path="/5387F9D3/53880A7F" Ref="R10"  Part="1"
-F 0 "R10" V 6330 2650 40  0000 C CNN
+AR Path="/5387F9D3/53880A7F" Ref="R4"  Part="1"
+AR Path="/539441D7/53880A7F" Ref="R16"  Part="1"
+F 0 "R4" V 6330 2650 40  0000 C CNN
 F 1 "R" V 6257 2651 40  0000 C CNN
 F 2 "~" V 6180 2650 30  0000 C CNN
@@
 U 1 1 53880A85
 P 6250 2850
-AR Path="/5387F99B/53880A85" Ref="R5"  Part="1"
-AR Path="/5387F9D3/53880A85" Ref="R11"  Part="1"
-F 0 "R11" V 6330 2850 40  0000 C CNN
+AR Path="/5387F9D3/53880A85" Ref="R5"  Part="1"
+AR Path="/539441D7/53880A85" Ref="R17"  Part="1"
+F 0 "R5" V 6330 2850 40  0000 C CNN
 F 1 "R" V 6257 2851 40  0000 C CNN
 F 2 "~" V 6180 2850 30  0000 C CNN
@@
 U 1 1 53880BE6
 P 7150 3450
-AR Path="/5387F99B/53880BE6" Ref="J3"  Part="1"
-AR Path="/5387F9D3/53880BE6" Ref="J5"  Part="1"
-F 0 "J5" H 7150 3700 60  0000 C CNN
+AR Path="/5387F9D3/53880BE6" Ref="J3"  Part="1"
+AR Path="/539441D7/53880BE6" Ref="J16"  Part="1"
+F 0 "J3" H 7150 3700 60  0000 C CNN
 F 1 "CONN_LED" H 7150 3200 60  0000 C CNN
 F 2 "~" H 7000 3400 60  0000 C CNN
@@
 U 1 1 53880BEC
 P 6250 3350
-AR Path="/5387F99B/53880BEC" Ref="R6"  Part="1"
-AR Path="/5387F9D3/53880BEC" Ref="R12"  Part="1"
-F 0 "R12" V 6330 3350 40  0000 C CNN
+AR Path="/5387F9D3/53880BEC" Ref="R6"  Part="1"
+AR Path="/539441D7/53880BEC" Ref="R18"  Part="1"
+F 0 "R6" V 6330 3350 40  0000 C CNN
 F 1 "R" V 6257 3351 40  0000 C CNN
 F 2 "~" V 6180 3350 30  0000 C CNN
@@
 U 1 1 53880BF2
 P 6250 3550
-AR Path="/5387F99B/53880BF2" Ref="R7"  Part="1"
-AR Path="/5387F9D3/53880BF2" Ref="R13"  Part="1"
-F 0 "R13" V 6330 3550 40  0000 C CNN
+AR Path="/5387F9D3/53880BF2" Ref="R7"  Part="1"
+AR Path="/539441D7/53880BF2" Ref="R19"  Part="1"
+F 0 "R7" V 6330 3550 40  0000 C CNN
 F 1 "R" V 6257 3551 40  0000 C CNN
 F 2 "~" V 6180 3550 30  0000 C CNN
@@
 U 1 1 53880BF8
 P 6250 3750
-AR Path="/5387F99B/53880BF8" Ref="R8"  Part="1"
-AR Path="/5387F9D3/53880BF8" Ref="R14"  Part="1"
-F 0 "R14" V 6330 3750 40  0000 C CNN
+AR Path="/5387F9D3/53880BF8" Ref="R8"  Part="1"
+AR Path="/539441D7/53880BF8" Ref="R20"  Part="1"
+F 0 "R8" V 6330 3750 40  0000 C CNN
 F 1 "R" V 6257 3751 40  0000 C CNN
 F 2 "~" V 6180 3750 30  0000 C CNN
@@
 U 1 1 53881290
 P 5300 3100
-AR Path="/5387F99B/53881290" Ref="U5"  Part="1"
-AR Path="/5387F9D3/53881290" Ref="U9"  Part="1"
-F 0 "U9" H 5300 3350 60  0000 C CNN
+AR Path="/5387F9D3/53881290" Ref="U5"  Part="1"
+AR Path="/539441D7/53881290" Ref="U15"  Part="1"
+F 0 "U5" H 5300 3350 60  0000 C CNN
 F 1 "AO4828" H 5300 2850 60  0000 C CNN
 F 2 "~" H 5250 2650 60  0000 C CNN
@@
 U 1 1 538812D6
 P 5300 2500
-AR Path="/5387F99B/538812D6" Ref="U4"  Part="1"
-AR Path="/5387F9D3/538812D6" Ref="U8"  Part="1"
-F 0 "U8" H 5300 2750 60  0000 C CNN
+AR Path="/5387F9D3/538812D6" Ref="U4"  Part="1"
+AR Path="/539441D7/538812D6" Ref="U14"  Part="1"
+F 0 "U4" H 5300 2750 60  0000 C CNN
 F 1 "AO4828" H 5300 2250 60  0000 C CNN
 F 2 "~" H 5250 2050 60  0000 C CNN
@@
 U 1 1 538812F1
 P 5300 3700
-AR Path="/5387F99B/538812F1" Ref="U6"  Part="1"
-AR Path="/5387F9D3/538812F1" Ref="U10"  Part="1"
-F 0 "U10" H 5300 3950 60  0000 C CNN
+AR Path="/5387F9D3/538812F1" Ref="U6"  Part="1"
+AR Path="/539441D7/538812F1" Ref="U16"  Part="1"
+F 0 "U6" H 5300 3950 60  0000 C CNN
 F 1 "AO4828" H 5300 3450 60  0000 C CNN
 F 2 "~" H 5250 3250 60  0000 C CNN
@@
 U 1 1 53881504
 P 4700 3450
-AR Path="/5387F99B/53881504" Ref="#PWR016"  Part="1"
-AR Path="/5387F9D3/53881504" Ref="#PWR023"  Part="1"
-F 0 "#PWR023" H 4700 3450 30  0001 C CNN
+AR Path="/5387F9D3/53881504" Ref="#PWR016"  Part="1"
+AR Path="/539441D7/53881504" Ref="#PWR077"  Part="1"
+F 0 "#PWR016" H 4700 3450 30  0001 C CNN
 F 1 "GND" H 4700 3380 30  0001 C CNN
 F 2 "" H 4700 3450 60  0000 C CNN
@@
 U 1 1 53881511
 P 4700 2850
-AR Path="/5387F99B/53881511" Ref="#PWR017"  Part="1"
-AR Path="/5387F9D3/53881511" Ref="#PWR024"  Part="1"
-F 0 "#PWR024" H 4700 2850 30  0001 C CNN
+AR Path="/5387F9D3/53881511" Ref="#PWR017"  Part="1"
+AR Path="/539441D7/53881511" Ref="#PWR078"  Part="1"
+F 0 "#PWR017" H 4700 2850 30  0001 C CNN
 F 1 "GND" H 4700 2780 30  0001 C CNN
 F 2 "" H 4700 2850 60  0000 C CNN
@@
 U 1 1 53881517
 P 4700 2250
-AR Path="/5387F99B/53881517" Ref="#PWR018"  Part="1"
-AR Path="/5387F9D3/53881517" Ref="#PWR025"  Part="1"
-F 0 "#PWR025" H 4700 2250 30  0001 C CNN
+AR Path="/5387F9D3/53881517" Ref="#PWR018"  Part="1"
+AR Path="/539441D7/53881517" Ref="#PWR079"  Part="1"
+F 0 "#PWR018" H 4700 2250 30  0001 C CNN
 F 1 "GND" H 4700 2180 30  0001 C CNN
 F 2 "" H 4700 2250 60  0000 C CNN
@@
 U 1 1 53881AE0
 P 3000 2800
-AR Path="/5387F99B/53881AE0" Ref="#PWR019"  Part="1"
-AR Path="/5387F9D3/53881AE0" Ref="#PWR026"  Part="1"
-F 0 "#PWR026" H 3000 2760 30  0001 C CNN
+AR Path="/5387F9D3/53881AE0" Ref="#PWR019"  Part="1"
+AR Path="/539441D7/53881AE0" Ref="#PWR080"  Part="1"
+F 0 "#PWR019" H 3000 2760 30  0001 C CNN
 F 1 "+3.3V" H 3000 2910 30  0000 C CNN
 F 2 "" H 3000 2800 60  0000 C CNN
@@
 U 1 1 53897F20
 P 3000 3650
-AR Path="/5387F99B/53897F20" Ref="#PWR020"  Part="1"
-AR Path="/5387F9D3/53897F20" Ref="#PWR027"  Part="1"
-F 0 "#PWR027" H 3000 3650 30  0001 C CNN
+AR Path="/5387F9D3/53897F20" Ref="#PWR020"  Part="1"
+AR Path="/539441D7/53897F20" Ref="#PWR081"  Part="1"
+F 0 "#PWR020" H 3000 3650 30  0001 C CNN
 F 1 "GND" H 3000 3580 30  0001 C CNN
 F 2 "" H 3000 3650 60  0000 C CNN
@@
 $EndComp
 Text HLabel 3000 3050 0    60   UnSpc ~ 0
-LED_SDOUT
+SDOUT
 Text HLabel 3000 2950 0    60   UnSpc ~ 0
-LED_SDIN
+SDIN
 Wire Wire Line
 	6650 2500 6500 2500
@@
 U 1 1 538B7495
 P 6250 2250
-AR Path="/5387F99B/538B7495" Ref="#PWR021"  Part="1"
-AR Path="/5387F9D3/538B7495" Ref="#PWR028"  Part="1"
-F 0 "#PWR028" H 6250 2220 20  0001 C CNN
+AR Path="/5387F9D3/538B7495" Ref="#PWR021"  Part="1"
+AR Path="/539441D7/538B7495" Ref="#PWR082"  Part="1"
+F 0 "#PWR021" H 6250 2220 20  0001 C CNN
 F 1 "+8V" H 6250 2360 30  0000 C CNN
 F 2 "" H 6250 2250 60  0000 C CNN
@@
 U 1 1 538B74AC
 P 6250 3150
-AR Path="/5387F99B/538B74AC" Ref="#PWR022"  Part="1"
-AR Path="/5387F9D3/538B74AC" Ref="#PWR029"  Part="1"
-F 0 "#PWR029" H 6250 3120 20  0001 C CNN
+AR Path="/5387F9D3/538B74AC" Ref="#PWR022"  Part="1"
+AR Path="/539441D7/538B74AC" Ref="#PWR083"  Part="1"
+F 0 "#PWR022" H 6250 3120 20  0001 C CNN
 F 1 "+8V" H 6250 3260 30  0000 C CNN
 F 2 "" H 6250 3150 60  0000 C CNN

Commit message: 
Parts:
- U3: value SHFTREG_H -> SN74HC595
Changed lines of the file:
@@
 $Descr A4 11693 8268
 encoding utf-8
-Sheet 3 15
+Sheet 15 15
 Title ""
 Date "8 jun 2014"
@@
 AR Path="/5387F9D3/53880946" Ref="U3"  Part="1"
 AR Path="/539441D7/53880946" Ref="U13"  Part="1"
-F 0 "U3" H 3600 3750 60  0000 C CNN
-F 1 "SHFTREG_H" H 3600 2650 60  0000 C CNN
+F 0 "U13" H 3600 3750 60  0000 C CNN
+F 1 "SN74HC595" H 3600 2650 60  0000 C CNN
 F 2 "~" V 3350 3300 60  0000 C CNN
 F 3 "~" V 3350 3300 60  0000 C CNN
@@
 AR Path="/5387F9D3/53880A57" Ref="J2"  Part="1"
 AR Path="/539441D7/53880A57" Ref="J15"  Part="1"
-F 0 "J2" H 7150 2800 60  0000 C CNN
+F 0 "J15" H 7150 2800 60  0000 C CNN
 F 1 "CONN_LED" H 7150 2300 60  0000 C CNN
 F 2 "~" H 7000 2500 60  0000 C CNN
@@
 AR Path="/5387F9D3/53880A79" Ref="R3"  Part="1"
 AR Path="/539441D7/53880A79" Ref="R15"  Part="1"
-F 0 "R3" V 6330 2450 40  0000 C CNN
+F 0 "R15" V 6330 2450 40  0000 C CNN
 F 1 "R" V 6257 2451 40  0000 C CNN
 F 2 "~" V 6180 2450 30  0000 C CNN
@@
 AR Path="/5387F9D3/53880A7F" Ref="R4"  Part="1"
 AR Path="/539441D7/53880A7F" Ref="R16"  Part="1"
-F 0 "R4" V 6330 2650 40  0000 C CNN
+F 0 "R16" V 6330 2650 40  0000 C CNN
 F 1 "R" V 6257 2651 40  0000 C CNN
 F 2 "~" V 6180 2650 30  0000 C CNN
@@
 AR Path="/5387F9D3/53880A85" Ref="R5"  Part="1"
 AR Path="/539441D7/53880A85" Ref="R17"  Part="1"
-F 0 "R5" V 6330 2850 40  0000 C CNN
+F 0 "R17" V 6330 2850 40  0000 C CNN
 F 1 "R" V 6257 2851 40  0000 C CNN
 F 2 "~" V 6180 2850 30  0000 C CNN
@@
 AR Path="/5387F9D3/53880BE6" Ref="J3"  Part="1"
 AR Path="/539441D7/53880BE6" Ref="J16"  Part="1"
-F 0 "J3" H 7150 3700 60  0000 C CNN
+F 0 "J16" H 7150 3700 60  0000 C CNN
 F 1 "CONN_LED" H 7150 3200 60  0000 C CNN
 F 2 "~" H 7000 3400 60  0000 C CNN
@@
 AR Path="/5387F9D3/53880BEC" Ref="R6"  Part="1"
 AR Path="/539441D7/53880BEC" Ref="R18"  Part="1"
-F 0 "R6" V 6330 3350 40  0000 C CNN
+F 0 "R18" V 6330 3350 40  0000 C CNN
 F 1 "R" V 6257 3351 40  0000 C CNN
 F 2 "~" V 6180 3350 30  0000 C CNN
@@
 AR Path="/5387F9D3/53880BF2" Ref="R7"  Part="1"
 AR Path="/539441D7/53880BF2" Ref="R19"  Part="1"
-F 0 "R7" V 6330 3550 40  0000 C CNN
+F 0 "R19" V 6330 3550 40  0000 C CNN
 F 1 "R" V 6257 3551 40  0000 C CNN
 F 2 "~" V 6180 3550 30  0000 C CNN
@@
 AR Path="/5387F9D3/53880BF8" Ref="R8"  Part="1"
 AR Path="/539441D7/53880BF8" Ref="R20"  Part="1"
-F 0 "R8" V 6330 3750 40  0000 C CNN
+F 0 "R20" V 6330 3750 40  0000 C CNN
 F 1 "R" V 6257 3751 40  0000 C CNN
 F 2 "~" V 6180 3750 30  0000 C CNN
@@
 AR Path="/5387F9D3/53881290" Ref="U5"  Part="1"
 AR Path="/539441D7/53881290" Ref="U15"  Part="1"
-F 0 "U5" H 5300 3350 60  0000 C CNN
+F 0 "U15" H 5300 3350 60  0000 C CNN
 F 1 "AO4828" H 5300 2850 60  0000 C CNN
 F 2 "~" H 5250 2650 60  0000 C CNN
@@
 AR Path="/5387F9D3/538812D6" Ref="U4"  Part="1"
 AR Path="/539441D7/538812D6" Ref="U14"  Part="1"
-F 0 "U4" H 5300 2750 60  0000 C CNN
+F 0 "U14" H 5300 2750 60  0000 C CNN
 F 1 "AO4828" H 5300 2250 60  0000 C CNN
 F 2 "~" H 5250 2050 60  0000 C CNN
@@
 AR Path="/5387F9D3/538812F1" Ref="U6"  Part="1"
 AR Path="/539441D7/538812F1" Ref="U16"  Part="1"
-F 0 "U6" H 5300 3950 60  0000 C CNN
+F 0 "U16" H 5300 3950 60  0000 C CNN
 F 1 "AO4828" H 5300 3450 60  0000 C CNN
 F 2 "~" H 5250 3250 60  0000 C CNN
@@
 AR Path="/5387F9D3/53881504" Ref="#PWR016"  Part="1"
 AR Path="/539441D7/53881504" Ref="#PWR077"  Part="1"
-F 0 "#PWR016" H 4700 3450 30  0001 C CNN
+F 0 "#PWR077" H 4700 3450 30  0001 C CNN
 F 1 "GND" H 4700 3380 30  0001 C CNN
 F 2 "" H 4700 3450 60  0000 C CNN
@@
 AR Path="/5387F9D3/53881511" Ref="#PWR017"  Part="1"
 AR Path="/539441D7/53881511" Ref="#PWR078"  Part="1"
-F 0 "#PWR017" H 4700 2850 30  0001 C CNN
+F 0 "#PWR078" H 4700 2850 30  0001 C CNN
 F 1 "GND" H 4700 2780 30  0001 C CNN
 F 2 "" H 4700 2850 60  0000 C CNN
@@
 AR Path="/5387F9D3/53881517" Ref="#PWR018"  Part="1"
 AR Path="/539441D7/53881517" Ref="#PWR079"  Part="1"
-F 0 "#PWR018" H 4700 2250 30  0001 C CNN
+F 0 "#PWR079" H 4700 2250 30  0001 C CNN
 F 1 "GND" H 4700 2180 30  0001 C CNN
 F 2 "" H 4700 2250 60  0000 C CNN
@@
 AR Path="/5387F9D3/53881AE0" Ref="#PWR019"  Part="1"
 AR Path="/539441D7/53881AE0" Ref="#PWR080"  Part="1"
-F 0 "#PWR019" H 3000 2760 30  0001 C CNN
+F 0 "#PWR080" H 3000 2760 30  0001 C CNN
 F 1 "+3.3V" H 3000 2910 30  0000 C CNN
 F 2 "" H 3000 2800 60  0000 C CNN
@@
 AR Path="/5387F9D3/53897F20" Ref="#PWR020"  Part="1"
 AR Path="/539441D7/53897F20" Ref="#PWR081"  Part="1"
-F 0 "#PWR020" H 3000 3650 30  0001 C CNN
+F 0 "#PWR081" H 3000 3650 30  0001 C CNN
 F 1 "GND" H 3000 3580 30  0001 C CNN
 F 2 "" H 3000 3650 60  0000 C CNN
@@
 AR Path="/5387F9D3/538B7495" Ref="#PWR021"  Part="1"
 AR Path="/539441D7/538B7495" Ref="#PWR082"  Part="1"
-F 0 "#PWR021" H 6250 2220 20  0001 C CNN
+F 0 "#PWR082" H 6250 2220 20  0001 C CNN
 F 1 "+8V" H 6250 2360 30  0000 C CNN
 F 2 "" H 6250 2250 60  0000 C CNN
@@
 AR Path="/5387F9D3/538B74AC" Ref="#PWR022"  Part="1"
 AR Path="/539441D7/538B74AC" Ref="#PWR083"  Part="1"
-F 0 "#PWR022" H 6250 3120 20  0001 C CNN
+F 0 "#PWR083" H 6250 3120 20  0001 C CNN
 F 1 "+8V" H 6250 3260 30  0000 C CNN
 F 2 "" H 6250 3150 60  0000 C CNN
