File: Kicad/LED_DUAL_DRIVER.sch (KiCad schematic (older format))
At the start: 12 parts, among them J2 CONN_LED, J3 CONN_LED, U3 SN74HC595, U4 AO4828, U5 AO4828, U6 AO4828

Commit message: 
Parts:
- R3, R6: value R -> 300
- R4, R5, R7, R8: value R -> 249
Changed lines of the file:
@@
 LIBS:contrib
 LIBS:valves
-LIBS:___power_diode
-LIBS:__batterybarlug
-LIBS:__freedom_x
-LIBS:__xbee-pro
-LIBS:CAR
 LIBS:car_v3-cache
 EELAYER 27 0
@@
 $Descr A4 11693 8268
 encoding utf-8
-Sheet 15 15
+Sheet 3 15
 Title ""
-Date "8 jun 2014"
+Date "13 jul 2014"
 Rev ""
 Comp ""
@@
 AR Path="/5387F9D3/53880946" Ref="U3"  Part="1"
 AR Path="/539441D7/53880946" Ref="U13"  Part="1"
-F 0 "U13" H 3600 3750 60  0000 C CNN
+F 0 "U3" H 3600 3750 60  0000 C CNN
 F 1 "SN74HC595" H 3600 2650 60  0000 C CNN
 F 2 "~" V 3350 3300 60  0000 C CNN
@@
 AR Path="/5387F9D3/53880A57" Ref="J2"  Part="1"
 AR Path="/539441D7/53880A57" Ref="J15"  Part="1"
-F 0 "J15" H 7150 2800 60  0000 C CNN
+F 0 "J2" H 7150 2800 60  0000 C CNN
 F 1 "CONN_LED" H 7150 2300 60  0000 C CNN
 F 2 "~" H 7000 2500 60  0000 C CNN
@@
 AR Path="/5387F9D3/53880A79" Ref="R3"  Part="1"
 AR Path="/539441D7/53880A79" Ref="R15"  Part="1"
-F 0 "R15" V 6330 2450 40  0000 C CNN
-F 1 "R" V 6257 2451 40  0000 C CNN
+F 0 "R3" V 6330 2450 40  0000 C CNN
+F 1 "300" V 6257 2451 40  0000 C CNN
 F 2 "~" V 6180 2450 30  0000 C CNN
 F 3 "~" H 6250 2450 30  0000 C CNN
@@
 AR Path="/5387F9D3/53880A7F" Ref="R4"  Part="1"
 AR Path="/539441D7/53880A7F" Ref="R16"  Part="1"
-F 0 "R16" V 6330 2650 40  0000 C CNN
-F 1 "R" V 6257 2651 40  0000 C CNN
+F 0 "R4" V 6330 2650 40  0000 C CNN
+F 1 "249" V 6257 2651 40  0000 C CNN
 F 2 "~" V 6180 2650 30  0000 C CNN
 F 3 "~" H 6250 2650 30  0000 C CNN
@@
 AR Path="/5387F9D3/53880A85" Ref="R5"  Part="1"
 AR Path="/539441D7/53880A85" Ref="R17"  Part="1"
-F 0 "R17" V 6330 2850 40  0000 C CNN
-F 1 "R" V 6257 2851 40  0000 C CNN
+F 0 "R5" V 6330 2850 40  0000 C CNN
+F 1 "249" V 6257 2851 40  0000 C CNN
 F 2 "~" V 6180 2850 30  0000 C CNN
 F 3 "~" H 6250 2850 30  0000 C CNN
@@
 AR Path="/5387F9D3/53880BE6" Ref="J3"  Part="1"
 AR Path="/539441D7/53880BE6" Ref="J16"  Part="1"
-F 0 "J16" H 7150 3700 60  0000 C CNN
+F 0 "J3" H 7150 3700 60  0000 C CNN
 F 1 "CONN_LED" H 7150 3200 60  0000 C CNN
 F 2 "~" H 7000 3400 60  0000 C CNN
@@
 AR Path="/5387F9D3/53880BEC" Ref="R6"  Part="1"
 AR Path="/539441D7/53880BEC" Ref="R18"  Part="1"
-F 0 "R18" V 6330 3350 40  0000 C CNN
-F 1 "R" V 6257 3351 40  0000 C CNN
+F 0 "R6" V 6330 3350 40  0000 C CNN
+F 1 "300" V 6257 3351 40  0000 C CNN
 F 2 "~" V 6180 3350 30  0000 C CNN
 F 3 "~" H 6250 3350 30  0000 C CNN
@@
 AR Path="/5387F9D3/53880BF2" Ref="R7"  Part="1"
 AR Path="/539441D7/53880BF2" Ref="R19"  Part="1"
-F 0 "R19" V 6330 3550 40  0000 C CNN
-F 1 "R" V 6257 3551 40  0000 C CNN
+F 0 "R7" V 6330 3550 40  0000 C CNN
+F 1 "249" V 6257 3551 40  0000 C CNN
 F 2 "~" V 6180 3550 30  0000 C CNN
 F 3 "~" H 6250 3550 30  0000 C CNN
@@
 AR Path="/5387F9D3/53880BF8" Ref="R8"  Part="1"
 AR Path="/539441D7/53880BF8" Ref="R20"  Part="1"
-F 0 "R20" V 6330 3750 40  0000 C CNN
-F 1 "R" V 6257 3751 40  0000 C CNN
+F 0 "R8" V 6330 3750 40  0000 C CNN
+F 1 "249" V 6257 3751 40  0000 C CNN
 F 2 "~" V 6180 3750 30  0000 C CNN
 F 3 "~" H 6250 3750 30  0000 C CNN
@@
 AR Path="/5387F9D3/53881290" Ref="U5"  Part="1"
 AR Path="/539441D7/53881290" Ref="U15"  Part="1"
-F 0 "U15" H 5300 3350 60  0000 C CNN
+F 0 "U5" H 5300 3350 60  0000 C CNN
 F 1 "AO4828" H 5300 2850 60  0000 C CNN
 F 2 "~" H 5250 2650 60  0000 C CNN
@@
 AR Path="/5387F9D3/538812D6" Ref="U4"  Part="1"
 AR Path="/539441D7/538812D6" Ref="U14"  Part="1"
-F 0 "U14" H 5300 2750 60  0000 C CNN
+F 0 "U4" H 5300 2750 60  0000 C CNN
 F 1 "AO4828" H 5300 2250 60  0000 C CNN
 F 2 "~" H 5250 2050 60  0000 C CNN
@@
 AR Path="/5387F9D3/538812F1" Ref="U6"  Part="1"
 AR Path="/539441D7/538812F1" Ref="U16"  Part="1"
-F 0 "U16" H 5300 3950 60  0000 C CNN
+F 0 "U6" H 5300 3950 60  0000 C CNN
 F 1 "AO4828" H 5300 3450 60  0000 C CNN
 F 2 "~" H 5250 3250 60  0000 C CNN
@@
 AR Path="/5387F9D3/53881504" Ref="#PWR016"  Part="1"
 AR Path="/539441D7/53881504" Ref="#PWR077"  Part="1"
-F 0 "#PWR077" H 4700 3450 30  0001 C CNN
+F 0 "#PWR016" H 4700 3450 30  0001 C CNN
 F 1 "GND" H 4700 3380 30  0001 C CNN
 F 2 "" H 4700 3450 60  0000 C CNN
@@
 AR Path="/5387F9D3/53881511" Ref="#PWR017"  Part="1"
 AR Path="/539441D7/53881511" Ref="#PWR078"  Part="1"
-F 0 "#PWR078" H 4700 2850 30  0001 C CNN
+F 0 "#PWR017" H 4700 2850 30  0001 C CNN
 F 1 "GND" H 4700 2780 30  0001 C CNN
 F 2 "" H 4700 2850 60  0000 C CNN
@@
 AR Path="/5387F9D3/53881517" Ref="#PWR018"  Part="1"
 AR Path="/539441D7/53881517" Ref="#PWR079"  Part="1"
-F 0 "#PWR079" H 4700 2250 30  0001 C CNN
+F 0 "#PWR018" H 4700 2250 30  0001 C CNN
 F 1 "GND" H 4700 2180 30  0001 C CNN
 F 2 "" H 4700 2250 60  0000 C CNN
@@
 AR Path="/5387F9D3/53881AE0" Ref="#PWR019"  Part="1"
 AR Path="/539441D7/53881AE0" Ref="#PWR080"  Part="1"
-F 0 "#PWR080" H 3000 2760 30  0001 C CNN
+F 0 "#PWR019" H 3000 2760 30  0001 C CNN
 F 1 "+3.3V" H 3000 2910 30  0000 C CNN
 F 2 "" H 3000 2800 60  0000 C CNN
@@
 AR Path="/5387F9D3/53897F20" Ref="#PWR020"  Part="1"
 AR Path="/539441D7/53897F20" Ref="#PWR081"  Part="1"
-F 0 "#PWR081" H 3000 3650 30  0001 C CNN
+F 0 "#PWR020" H 3000 3650 30  0001 C CNN
 F 1 "GND" H 3000 3580 30  0001 C CNN
 F 2 "" H 3000 3650 60  0000 C CNN
@@
 AR Path="/5387F9D3/538B7495" Ref="#PWR021"  Part="1"
 AR Path="/539441D7/538B7495" Ref="#PWR082"  Part="1"
-F 0 "#PWR082" H 6250 2220 20  0001 C CNN
+F 0 "#PWR021" H 6250 2220 20  0001 C CNN
 F 1 "+8V" H 6250 2360 30  0000 C CNN
 F 2 "" H 6250 2250 60  0000 C CNN
@@
 AR Path="/5387F9D3/538B74AC" Ref="#PWR022"  Part="1"
 AR Path="/539441D7/538B74AC" Ref="#PWR083"  Part="1"
-F 0 "#PWR083" H 6250 3120 20  0001 C CNN
+F 0 "#PWR022" H 6250 3120 20  0001 C CNN
 F 1 "+8V" H 6250 3260 30  0000 C CNN
 F 2 "" H 6250 3150 60  0000 C CNN
