File: Kicad/BATTERY.sch (KiCad schematic (older format))
At the start: 3 parts, among them J9 CONN2

Commit message: 
Parts:
- removed L5: __BATTERYBARLUG, ~, symbol __BATTERYBARLUG
- added L2: LUG, ~, symbol LUG
- renumbered J9 to J6
Changed lines of the file:
@@
 $Descr A4 11693 8268
 encoding utf-8
-Sheet 13 15
+Sheet 10 15
 Title ""
-Date "1 jun 2014"
+Date "7 jun 2014"
 Rev ""
 Comp ""
@@
 $EndDescr
 $Comp
-L CONN2 J9
+L CONN2 J6
 U 1 1 53880043
 P 6550 3650
-AR Path="/5387FDA2/53880043" Ref="J9"  Part="1"
-AR Path="/5387FDCE/53880043" Ref="J10"  Part="1"
-AR Path="/5387FDE3/53880043" Ref="J11"  Part="1"
-AR Path="/5387FE00/53880043" Ref="J12"  Part="1"
-AR Path="/5387FE16/53880043" Ref="J13"  Part="1"
-AR Path="/5387FE2E/53880043" Ref="J14"  Part="1"
-F 0 "J9" H 6550 3850 60  0000 C CNN
+AR Path="/5387FDA2/53880043" Ref="J6"  Part="1"
+AR Path="/5387FDCE/53880043" Ref="J7"  Part="1"
+AR Path="/5387FDE3/53880043" Ref="J8"  Part="1"
+AR Path="/5387FE00/53880043" Ref="J9"  Part="1"
+AR Path="/5387FE16/53880043" Ref="J10"  Part="1"
+AR Path="/5387FE2E/53880043" Ref="J11"  Part="1"
+F 0 "J11" H 6550 3850 60  0000 C CNN
 F 1 "CONN2" H 6550 3450 60  0000 C CNN
 F 2 "~" H 6400 3650 60  0000 C CNN
@@
 $EndComp
 $Comp
-L GND #PWR058
+L GND #PWR033
 U 1 1 53880055
 P 6100 3850
-AR Path="/5387FDA2/53880055" Ref="#PWR058"  Part="1"
-AR Path="/5387FDCE/53880055" Ref="#PWR060"  Part="1"
-AR Path="/5387FDE3/53880055" Ref="#PWR062"  Part="1"
-AR Path="/5387FE00/53880055" Ref="#PWR064"  Part="1"
-AR Path="/5387FE16/53880055" Ref="#PWR066"  Part="1"
-AR Path="/5387FE2E/53880055" Ref="#PWR068"  Part="1"
-F 0 "#PWR058" H 6100 3850 30  0001 C CNN
+AR Path="/5387FDA2/53880055" Ref="#PWR033"  Part="1"
+AR Path="/5387FDCE/53880055" Ref="#PWR035"  Part="1"
+AR Path="/5387FDE3/53880055" Ref="#PWR037"  Part="1"
+AR Path="/5387FE00/53880055" Ref="#PWR039"  Part="1"
+AR Path="/5387FE16/53880055" Ref="#PWR041"  Part="1"
+AR Path="/5387FE2E/53880055" Ref="#PWR043"  Part="1"
+F 0 "#PWR043" H 6100 3850 30  0001 C CNN
 F 1 "GND" H 6100 3780 30  0001 C CNN
 F 2 "" H 6100 3850 60  0000 C CNN
@@
 AR Path="/5387FE16/538800B9" Ref="D5"  Part="1"
 AR Path="/5387FE2E/538800B9" Ref="D6"  Part="1"
-F 0 "D1" H 5900 3650 40  0000 C CNN
+F 0 "D6" H 5900 3650 40  0000 C CNN
 F 1 "___POWER_DIODE" H 5900 3450 40  0000 C CNN
 F 2 "~" H 5900 3550 60  0000 C CNN
@@
 	1    5900 3550
 	-1   0    0    1
-$EndComp
-$Comp
-L __BATTERYBARLUG L5
-U 1 1 5388012D
-P 5350 3400
-AR Path="/5387FDA2/5388012D" Ref="L5"  Part="1"
-AR Path="/5387FDCE/5388012D" Ref="L6"  Part="1"
-AR Path="/5387FDE3/5388012D" Ref="L7"  Part="1"
-AR Path="/5387FE00/5388012D" Ref="L8"  Part="1"
-AR Path="/5387FE16/5388012D" Ref="L9"  Part="1"
-AR Path="/5387FE2E/5388012D" Ref="L10"  Part="1"
-F 0 "L5" H 5500 3350 60  0000 C CNN
-F 1 "__BATTERYBARLUG" H 5350 3450 20  0000 C CNN
-F 2 "~" H 5350 3450 60  0000 C CNN
-F 3 "~" H 5350 3450 60  0000 C CNN
-	1    5350 3400
-	1    0    0    -1
 $EndComp
 Wire Wire Line
@@
 Connection ~ 5350 3550
 $Comp
-L +8V #PWR067
-U 1 1 538B7656
+L LUG L2
+U 1 1 538B729A
+P 5350 3100
+AR Path="/5387FDA2/538B729A" Ref="L2"  Part="1"
+AR Path="/5387FDCE/538B729A" Ref="L3"  Part="1"
+AR Path="/5387FDE3/538B729A" Ref="L4"  Part="1"
+AR Path="/5387FE00/538B729A" Ref="L5"  Part="1"
+AR Path="/5387FE16/538B729A" Ref="L6"  Part="1"
+AR Path="/5387FE2E/538B729A" Ref="L7"  Part="1"
+F 0 "L7" H 5450 3100 60  0000 C CNN
+F 1 "LUG" H 5350 3200 20  0000 C CNN
+F 2 "~" H 5250 3050 60  0000 C CNN
+F 3 "~" H 5250 3050 60  0000 C CNN
+	1    5350 3100
+	1    0    0    -1
+$EndComp
+$Comp
+L +8V #PWR034
+U 1 1 538B73EC
 P 5150 3550
-AR Path="/5387FE16/538B7656" Ref="#PWR067"  Part="1"
-AR Path="/5387FDA2/538B7656" Ref="#PWR059"  Part="1"
-AR Path="/5387FDCE/538B7656" Ref="#PWR061"  Part="1"
-AR Path="/5387FDE3/538B7656" Ref="#PWR063"  Part="1"
-AR Path="/5387FE00/538B7656" Ref="#PWR065"  Part="1"
-AR Path="/5387FE2E/538B7656" Ref="#PWR069"  Part="1"
-F 0 "#PWR059" H 5150 3520 20  0001 C CNN
+AR Path="/5387FDA2/538B73EC" Ref="#PWR034"  Part="1"
+AR Path="/5387FDCE/538B73EC" Ref="#PWR036"  Part="1"
+AR Path="/5387FDE3/538B73EC" Ref="#PWR038"  Part="1"
+AR Path="/5387FE00/538B73EC" Ref="#PWR040"  Part="1"
+AR Path="/5387FE16/538B73EC" Ref="#PWR042"  Part="1"
+AR Path="/5387FE2E/538B73EC" Ref="#PWR044"  Part="1"
+F 0 "#PWR044" H 5150 3520 20  0001 C CNN
 F 1 "+8V" H 5150 3660 30  0000 C CNN
 F 2 "" H 5150 3550 60  0000 C CNN

Commit message: All wired. ERC passes with no errors. Might be good to go.
Parts:
- renumbered J6 to J4
Changed lines of the file:
@@
 Sheet 10 15
 Title ""
-Date "7 jun 2014"
+Date "8 jun 2014"
 Rev ""
 Comp ""
@@
 $EndDescr
 $Comp
-L CONN2 J6
+L CONN2 J4
 U 1 1 53880043
 P 6550 3650
-AR Path="/5387FDA2/53880043" Ref="J6"  Part="1"
-AR Path="/5387FDCE/53880043" Ref="J7"  Part="1"
-AR Path="/5387FDE3/53880043" Ref="J8"  Part="1"
-AR Path="/5387FE00/53880043" Ref="J9"  Part="1"
-AR Path="/5387FE16/53880043" Ref="J10"  Part="1"
-AR Path="/5387FE2E/53880043" Ref="J11"  Part="1"
-F 0 "J11" H 6550 3850 60  0000 C CNN
+AR Path="/5387FDA2/53880043" Ref="J4"  Part="1"
+AR Path="/5387FDCE/53880043" Ref="J5"  Part="1"
+AR Path="/5387FDE3/53880043" Ref="J6"  Part="1"
+AR Path="/5387FE00/53880043" Ref="J7"  Part="1"
+AR Path="/5387FE16/53880043" Ref="J8"  Part="1"
+AR Path="/5387FE2E/53880043" Ref="J9"  Part="1"
+F 0 "J9" H 6550 3850 60  0000 C CNN
 F 1 "CONN2" H 6550 3450 60  0000 C CNN
 F 2 "~" H 6400 3650 60  0000 C CNN
@@
 $EndComp
 $Comp
-L GND #PWR033
+L GND #PWR026
 U 1 1 53880055
 P 6100 3850
-AR Path="/5387FDA2/53880055" Ref="#PWR033"  Part="1"
-AR Path="/5387FDCE/53880055" Ref="#PWR035"  Part="1"
-AR Path="/5387FDE3/53880055" Ref="#PWR037"  Part="1"
-AR Path="/5387FE00/53880055" Ref="#PWR039"  Part="1"
-AR Path="/5387FE16/53880055" Ref="#PWR041"  Part="1"
-AR Path="/5387FE2E/53880055" Ref="#PWR043"  Part="1"
-F 0 "#PWR043" H 6100 3850 30  0001 C CNN
+AR Path="/5387FDA2/53880055" Ref="#PWR026"  Part="1"
+AR Path="/5387FDCE/53880055" Ref="#PWR028"  Part="1"
+AR Path="/5387FDE3/53880055" Ref="#PWR030"  Part="1"
+AR Path="/5387FE00/53880055" Ref="#PWR032"  Part="1"
+AR Path="/5387FE16/53880055" Ref="#PWR034"  Part="1"
+AR Path="/5387FE2E/53880055" Ref="#PWR036"  Part="1"
+F 0 "#PWR036" H 6100 3850 30  0001 C CNN
 F 1 "GND" H 6100 3780 30  0001 C CNN
 F 2 "" H 6100 3850 60  0000 C CNN
@@
 $EndComp
 $Comp
-L +8V #PWR034
+L +8V #PWR027
 U 1 1 538B73EC
 P 5150 3550
-AR Path="/5387FDA2/538B73EC" Ref="#PWR034"  Part="1"
-AR Path="/5387FDCE/538B73EC" Ref="#PWR036"  Part="1"
-AR Path="/5387FDE3/538B73EC" Ref="#PWR038"  Part="1"
-AR Path="/5387FE00/538B73EC" Ref="#PWR040"  Part="1"
-AR Path="/5387FE16/538B73EC" Ref="#PWR042"  Part="1"
-AR Path="/5387FE2E/538B73EC" Ref="#PWR044"  Part="1"
-F 0 "#PWR044" H 5150 3520 20  0001 C CNN
+AR Path="/5387FDA2/538B73EC" Ref="#PWR027"  Part="1"
+AR Path="/5387FDCE/538B73EC" Ref="#PWR029"  Part="1"
+AR Path="/5387FDE3/538B73EC" Ref="#PWR031"  Part="1"
+AR Path="/5387FE00/538B73EC" Ref="#PWR033"  Part="1"
+AR Path="/5387FE16/538B73EC" Ref="#PWR035"  Part="1"
+AR Path="/5387FE2E/538B73EC" Ref="#PWR037"  Part="1"
+F 0 "#PWR037" H 5150 3520 20  0001 C CNN
 F 1 "+8V" H 5150 3660 30  0000 C CNN
 F 2 "" H 5150 3550 60  0000 C CNN

Commit message: 
Parts:
- D1: value ___POWER_DIODE -> POWER_DIODE
Changed lines of the file:
@@
 LIBS:contrib
 LIBS:valves
-LIBS:___power_diode
-LIBS:__batterybarlug
-LIBS:__freedom_x
-LIBS:__xbee-pro
-LIBS:CAR
 LIBS:car_v3-cache
 EELAYER 27 0
@@
 $Descr A4 11693 8268
 encoding utf-8
-Sheet 10 15
+Sheet 9 15
 Title ""
-Date "8 jun 2014"
+Date "13 jul 2014"
 Rev ""
 Comp ""
@@
 AR Path="/5387FE2E/538800B9" Ref="D6"  Part="1"
 F 0 "D6" H 5900 3650 40  0000 C CNN
-F 1 "___POWER_DIODE" H 5900 3450 40  0000 C CNN
+F 1 "POWER_DIODE" H 5900 3450 40  0000 C CNN
 F 2 "~" H 5900 3550 60  0000 C CNN
 F 3 "~" H 5900 3550 60  0000 C CNN
