File: Kicad/MOTOR_DRIVER.sch (KiCad schematic (older format))
At the start: 8 parts, among them J4 CONN_MOTOR, U7 SHFTREG_H, U8 LV8727

Commit message: 
Parts:
- renumbered C7 to C1, C8 to C2, J4 to J1, L4 to L1, R7 to R1, R8 to R2, U7 to U1, U8 to U2
Connections:
- wire segments 49 -> 48
Changed lines of the file:
@@
 $EndDescr
 $Comp
-L LV8727 U8
+L LV8727 U2
 U 1 1 53880645
 P 5650 2400
-AR Path="/5387F7BE/53880645" Ref="U8"  Part="1"
 AR Path="/5387F728/53880645" Ref="U2"  Part="1"
 AR Path="/5387F76A/53880645" Ref="U4"  Part="1"
 AR Path="/5387F799/53880645" Ref="U6"  Part="1"
+AR Path="/5387F7BE/53880645" Ref="U8"  Part="1"
 F 0 "U2" V 4300 2600 60  0000 C CNN
 F 1 "LV8727" V 7050 2600 60  0000 C CNN
@@
 $EndComp
 $Comp
-L SHFTREG_H U7
+L SHFTREG_H U1
 U 1 1 53880692
 P 4250 5150
-AR Path="/5387F7BE/53880692" Ref="U7"  Part="1"
 AR Path="/5387F728/53880692" Ref="U1"  Part="1"
 AR Path="/5387F76A/53880692" Ref="U3"  Part="1"
 AR Path="/5387F799/53880692" Ref="U5"  Part="1"
+AR Path="/5387F7BE/53880692" Ref="U7"  Part="1"
 F 0 "U1" H 4250 5700 60  0000 C CNN
 F 1 "SHFTREG_H" H 4250 4600 60  0000 C CNN
@@
 $EndComp
 $Comp
-L __BATTERYBARLUG L4
+L __BATTERYBARLUG L1
 U 1 1 53880889
 P 4650 3900
-AR Path="/5387F7BE/53880889" Ref="L4"  Part="1"
 AR Path="/5387F728/53880889" Ref="L1"  Part="1"
 AR Path="/5387F76A/53880889" Ref="L2"  Part="1"
 AR Path="/5387F799/53880889" Ref="L3"  Part="1"
+AR Path="/5387F7BE/53880889" Ref="L4"  Part="1"
 F 0 "L1" H 4800 3850 60  0000 C CNN
 F 1 "__BATTERYBARLUG" H 4650 3950 20  0000 C CNN
@@
 $EndComp
 $Comp
-L R R8
+L R R2
 U 1 1 538A3F7A
 P 6750 2950
-AR Path="/5387F7BE/538A3F7A" Ref="R8"  Part="1"
 AR Path="/5387F728/538A3F7A" Ref="R2"  Part="1"
 AR Path="/5387F76A/538A3F7A" Ref="R4"  Part="1"
 AR Path="/5387F799/538A3F7A" Ref="R6"  Part="1"
+AR Path="/5387F7BE/538A3F7A" Ref="R8"  Part="1"
 F 0 "R2" V 6830 2950 40  0000 C CNN
 F 1 "0.1" V 6757 2951 40  0000 C CNN
@@
 $EndComp
 $Comp
-L R R7
+L R R1
 U 1 1 538A3F87
 P 4550 2950
-AR Path="/5387F7BE/538A3F87" Ref="R7"  Part="1"
 AR Path="/5387F728/538A3F87" Ref="R1"  Part="1"
 AR Path="/5387F76A/538A3F87" Ref="R3"  Part="1"
 AR Path="/5387F799/538A3F87" Ref="R5"  Part="1"
+AR Path="/5387F7BE/538A3F87" Ref="R7"  Part="1"
 F 0 "R1" V 4630 2950 40  0000 C CNN
 F 1 "0.1" V 4557 2951 40  0000 C CNN
@@
 $EndComp
 $Comp
-L C C7
+L C C1
 U 1 1 538A3FA9
 P 4850 4350
-AR Path="/5387F7BE/538A3FA9" Ref="C7"  Part="1"
 AR Path="/5387F728/538A3FA9" Ref="C1"  Part="1"
 AR Path="/5387F76A/538A3FA9" Ref="C3"  Part="1"
 AR Path="/5387F799/538A3FA9" Ref="C5"  Part="1"
+AR Path="/5387F7BE/538A3FA9" Ref="C7"  Part="1"
 F 0 "C1" H 4850 4450 40  0000 L CNN
 F 1 "1000u" H 4856 4265 40  0000 L CNN
@@
 $EndComp
 $Comp
-L GND #PWR032
+L GND #PWR05
 U 1 1 538A3FB8
 P 4850 4600
-AR Path="/5387F7BE/538A3FB8" Ref="#PWR032"  Part="1"
 AR Path="/5387F728/538A3FB8" Ref="#PWR05"  Part="1"
 AR Path="/5387F76A/538A3FB8" Ref="#PWR014"  Part="1"
 AR Path="/5387F799/538A3FB8" Ref="#PWR023"  Part="1"
-F 0 "#PWR05" H 4850 4600 30  0001 C CNN
+AR Path="/5387F7BE/538A3FB8" Ref="#PWR032"  Part="1"
+F 0 "#PWR032" H 4850 4600 30  0001 C CNN
 F 1 "GND" H 4850 4530 30  0001 C CNN
 F 2 "" H 4850 4600 60  0000 C CNN
@@
 Connection ~ 4850 4050
 $Comp
-L GND #PWR033
+L GND #PWR06
 U 1 1 538A3FEF
 P 6350 2750
-AR Path="/5387F7BE/538A3FEF" Ref="#PWR033"  Part="1"
 AR Path="/5387F728/538A3FEF" Ref="#PWR06"  Part="1"
 AR Path="/5387F76A/538A3FEF" Ref="#PWR015"  Part="1"
 AR Path="/5387F799/538A3FEF" Ref="#PWR024"  Part="1"
-F 0 "#PWR06" H 6350 2750 30  0001 C CNN
+AR Path="/5387F7BE/538A3FEF" Ref="#PWR033"  Part="1"
+F 0 "#PWR033" H 6350 2750 30  0001 C CNN
 F 1 "GND" H 6350 2680 30  0001 C CNN
 F 2 "" H 6350 2750 60  0000 C CNN
@@
 $EndComp
 $Comp
-L GND #PWR034
+L GND #PWR07
 U 1 1 538A3FF5
 P 6650 2750
-AR Path="/5387F7BE/538A3FF5" Ref="#PWR034"  Part="1"
 AR Path="/5387F728/538A3FF5" Ref="#PWR07"  Part="1"
 AR Path="/5387F76A/538A3FF5" Ref="#PWR016"  Part="1"
 AR Path="/5387F799/538A3FF5" Ref="#PWR025"  Part="1"
-F 0 "#PWR07" H 6650 2750 30  0001 C CNN
+AR Path="/5387F7BE/538A3FF5" Ref="#PWR034"  Part="1"
+F 0 "#PWR034" H 6650 2750 30  0001 C CNN
 F 1 "GND" H 6650 2680 30  0001 C CNN
 F 2 "" H 6650 2750 60  0000 C CNN
@@
 $EndComp
 $Comp
-L GND #PWR035
+L GND #PWR08
 U 1 1 538A3FFB
 P 4650 2750
-AR Path="/5387F7BE/538A3FFB" Ref="#PWR035"  Part="1"
 AR Path="/5387F728/538A3FFB" Ref="#PWR08"  Part="1"
 AR Path="/5387F76A/538A3FFB" Ref="#PWR017"  Part="1"
 AR Path="/5387F799/538A3FFB" Ref="#PWR026"  Part="1"
-F 0 "#PWR08" H 4650 2750 30  0001 C CNN
+AR Path="/5387F7BE/538A3FFB" Ref="#PWR035"  Part="1"
+F 0 "#PWR035" H 4650 2750 30  0001 C CNN
 F 1 "GND" H 4650 2680 30  0001 C CNN
 F 2 "" H 4650 2750 60  0000 C CNN
@@
 Text HLabel 5650 2800 3    60   UnSpc ~ 0
 MOTOR_STEP
-Text HLabel 5550 2800 3    60   UnSpc ~ 0
+Text HLabel 5550 2700 3    60   UnSpc ~ 0
 MOTOR_FR
 $Comp
-L GND #PWR036
+L GND #PWR09
 U 1 1 538A4FB3
 P 4550 3250
-AR Path="/5387F7BE/538A4FB3" Ref="#PWR036"  Part="1"
 AR Path="/5387F728/538A4FB3" Ref="#PWR09"  Part="1"
 AR Path="/5387F76A/538A4FB3" Ref="#PWR018"  Part="1"
 AR Path="/5387F799/538A4FB3" Ref="#PWR027"  Part="1"
-F 0 "#PWR09" H 4550 3250 30  0001 C CNN
+AR Path="/5387F7BE/538A4FB3" Ref="#PWR036"  Part="1"
+F 0 "#PWR036" H 4550 3250 30  0001 C CNN
 F 1 "GND" H 4550 3180 30  0001 C CNN
 F 2 "" H 4550 3250 60  0000 C CNN
@@
 $EndComp
 $Comp
-L GND #PWR037
+L GND #PWR010
 U 1 1 538A4FB9
 P 6750 3250
-AR Path="/5387F7BE/538A4FB9" Ref="#PWR037"  Part="1"
 AR Path="/5387F728/538A4FB9" Ref="#PWR010"  Part="1"
 AR Path="/5387F76A/538A4FB9" Ref="#PWR019"  Part="1"
 AR Path="/5387F799/538A4FB9" Ref="#PWR028"  Part="1"
-F 0 "#PWR010" H 6750 3250 30  0001 C CNN
+AR Path="/5387F7BE/538A4FB9" Ref="#PWR037"  Part="1"
+F 0 "#PWR037" H 6750 3250 30  0001 C CNN
 F 1 "GND" H 6750 3180 30  0001 C CNN
 F 2 "" H 6750 3250 60  0000 C CNN
@@
 	6250 2700 6250 2800
 $Comp
-L C C8
+L C C2
 U 1 1 538A522E
 P 5800 3000
-AR Path="/5387F7BE/538A522E" Ref="C8"  Part="1"
 AR Path="/5387F728/538A522E" Ref="C2"  Part="1"
 AR Path="/5387F76A/538A522E" Ref="C4"  Part="1"
 AR Path="/5387F799/538A522E" Ref="C6"  Part="1"
+AR Path="/5387F7BE/538A522E" Ref="C8"  Part="1"
 F 0 "C2" H 5800 3100 40  0000 L CNN
 F 1 "180p" H 5806 2915 40  0000 L CNN
@@
 	5750 2800 5800 2800
 $Comp
-L GND #PWR038
+L GND #PWR011
 U 1 1 538A5251
 P 5800 3250
-AR Path="/5387F7BE/538A5251" Ref="#PWR038"  Part="1"
 AR Path="/5387F728/538A5251" Ref="#PWR011"  Part="1"
 AR Path="/5387F76A/538A5251" Ref="#PWR020"  Part="1"
 AR Path="/5387F799/538A5251" Ref="#PWR029"  Part="1"
-F 0 "#PWR011" H 5800 3250 30  0001 C CNN
+AR Path="/5387F7BE/538A5251" Ref="#PWR038"  Part="1"
+F 0 "#PWR038" H 5800 3250 30  0001 C CNN
 F 1 "GND" H 5800 3180 30  0001 C CNN
 F 2 "" H 5800 3250 60  0000 C CNN
@@
 NoConn ~ 4850 5500
 $Comp
-L CONN_MOTOR J4
+L CONN_MOTOR J1
 U 1 1 538A7481
 P 5850 1200
-AR Path="/5387F7BE/538A7481" Ref="J4"  Part="1"
 AR Path="/5387F728/538A7481" Ref="J1"  Part="1"
 AR Path="/5387F76A/538A7481" Ref="J2"  Part="1"
 AR Path="/5387F799/538A7481" Ref="J3"  Part="1"
+AR Path="/5387F7BE/538A7481" Ref="J4"  Part="1"
 F 0 "J1" H 5850 1350 60  0000 C CNN
 F 1 "CONN_MOTOR" H 6350 1200 60  0000 C CNN
@@
 	4950 4800 4850 4800
 $Comp
-L +3.3V #PWR039
+L +3.3V #PWR012
 U 1 1 538A78DB
 P 3650 4750
-AR Path="/5387F7BE/538A78DB" Ref="#PWR039"  Part="1"
 AR Path="/5387F728/538A78DB" Ref="#PWR012"  Part="1"
 AR Path="/5387F76A/538A78DB" Ref="#PWR021"  Part="1"
 AR Path="/5387F799/538A78DB" Ref="#PWR030"  Part="1"
-F 0 "#PWR012" H 3650 4710 30  0001 C CNN
+AR Path="/5387F7BE/538A78DB" Ref="#PWR039"  Part="1"
+F 0 "#PWR039" H 3650 4710 30  0001 C CNN
 F 1 "+3.3V" H 3650 4860 30  0000 C CNN
 F 2 "" H 3650 4750 60  0000 C CNN
@@
 	3650 4750 3650 4800
 $Comp
-L GND #PWR040
+L GND #PWR013
 U 1 1 538A7924
 P 3650 5600
-AR Path="/5387F7BE/538A7924" Ref="#PWR040"  Part="1"
 AR Path="/5387F728/538A7924" Ref="#PWR013"  Part="1"
 AR Path="/5387F76A/538A7924" Ref="#PWR022"  Part="1"
 AR Path="/5387F799/538A7924" Ref="#PWR031"  Part="1"
-F 0 "#PWR013" H 3650 5600 30  0001 C CNN
+AR Path="/5387F7BE/538A7924" Ref="#PWR040"  Part="1"
+F 0 "#PWR040" H 3650 5600 30  0001 C CNN
 F 1 "GND" H 3650 5530 30  0001 C CNN
 F 2 "" H 3650 5600 60  0000 C CNN
@@
 Wire Wire Line
 	5650 2700 5650 2800
-Wire Wire Line
-	5550 2700 5550 2800
 $EndSCHEMATC
