File: Kicad/XBEE.sch (KiCad schematic (older format))
At the start: 1 part, among them M1 __XBEE-PRO

Commit message: 
Connections:
- net XBEE_ON renamed ON
- net XBEE_RESET_b renamed RESET_b
- net XBEE_RX renamed RX
- net XBEE_TX renamed TX
Changed lines of the file:
@@
 $Descr A4 11693 8268
 encoding utf-8
-Sheet 8 15
+Sheet 5 15
 Title ""
-Date "1 jun 2014"
+Date "7 jun 2014"
 Rev ""
 Comp ""
@@
 $EndComp
 $Comp
-L GND #PWR055
+L GND #PWR030
 U 1 1 5389890A
 P 4950 4450
-F 0 "#PWR055" H 4950 4450 30  0001 C CNN
+F 0 "#PWR030" H 4950 4450 30  0001 C CNN
 F 1 "GND" H 4950 4380 30  0001 C CNN
 F 2 "" H 4950 4450 60  0000 C CNN
@@
 	4950 4450 4950 4350
 $Comp
-L +3.3V #PWR056
+L +3.3V #PWR031
 U 1 1 5389891E
 P 4950 2950
-F 0 "#PWR056" H 4950 2910 30  0001 C CNN
+F 0 "#PWR031" H 4950 2910 30  0001 C CNN
 F 1 "+3.3V" H 4950 3060 30  0000 C CNN
 F 2 "" H 4950 2950 60  0000 C CNN
@@
 NoConn ~ 6650 3600
 $Comp
-L +3.3V #PWR057
+L +3.3V #PWR032
 U 1 1 53898952
 P 6750 3850
-F 0 "#PWR057" H 6750 3810 30  0001 C CNN
+F 0 "#PWR032" H 6750 3810 30  0001 C CNN
 F 1 "+3.3V" H 6750 3960 30  0000 C CNN
 F 2 "" H 6750 3850 60  0000 C CNN
@@
 NoConn ~ 4950 4200
 Text HLabel 6700 4050 2    60   UnSpc ~ 0
-XBEE_ON
+ON
 Text HLabel 4900 3600 0    60   UnSpc ~ 0
-XBEE_RESET_b
+RESET_b
 Text HLabel 4900 3150 0    60   UnSpc ~ 0
-XBEE_RX
+RX
 Text HLabel 4900 3300 0    60   UnSpc ~ 0
-XBEE_TX
+TX
 Wire Wire Line
 	4900 3300 4950 3300

Commit message: 
Parts:
- M1: value __XBEE-PRO -> XBEE
Changed lines of the file:
@@
 P 5750 3700
 F 0 "M1" H 5450 4850 50  0000 L BNN
-F 1 "__XBEE-PRO" H 5550 2750 50  0000 L BNN
+F 1 "XBEE" H 5700 2750 50  0000 L BNN
 F 2 "xbee_r1-XBEE-PRO" H 5850 2900 50  0001 C CNN
 F 3 "~" H 5750 3700 60  0000 C CNN
