File: Kicad/car_v3.kicad_pcb (KiCad board)
At the start: 2 copper layers, 200 x 160 mm, 77 parts, among them J1 CONN_MOTOR, J10 FRDM_KL46Z, J11 FRDM_KL46Z, J12 CONN_MOTOR, J13 CONN_MOTOR, J14 CONN_MOTOR, J15 CONN_LED, J16 CONN_LED, J2 CONN_LED, J3 CONN_LED, J4 CONN2, J5 CONN2, J6 CONN2, J7 CONN2, J8 CONN2, J9 CONN2, M1 XBEE, U1 SN74HC595, U10 LV8727, U11 SN74HC595, U12 LV8727, U13 SN74HC595, U14 AO4828, U15 AO4828, U16 AO4828, U2 LV8727, U3 SN74HC595, U4 AO4828, U5 AO4828, U6 AO4828, U7 SN74HC595, U8 LV8727, U9 SN74HC595

Commit message: 
Parts:
- R3, R4, R5: moved to B.Cu
- moved J15 135.5 mm to (113.5, 193.5)
- moved R15 135.5 mm to (106.0, 197.5)
- moved R16 135.5 mm to (106.0, 193.5)
- moved R17 135.5 mm to (106.0, 189.5)
- moved J16 129.0 mm to (113.5, 53.0)
- moved R18 129.0 mm to (106.0, 57.0)
- moved R19 129.0 mm to (106.0, 53.0)
- moved R20 129.0 mm to (106.0, 49.0)
- moved J10 124.4 mm to (20.0, 164.0)
- moved J1 100.5 mm to (20.0, 53.0), turned to 270 degrees
- moved C6 74.2 mm to (242.5, 1.50)
- moved R11 74.2 mm to (232.5, -24.5)
- moved R12 74.2 mm to (242.5, 6.50)
- moved U3 73.2 mm to (170.5, 132.5)
- moved C5 65.8 mm to (201.0, 88.0), turned to 0 degrees
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
Commit message: 
Parts:
- removed J10: FRDM_KL46Z, __Freedom
- R6, R7, R8: moved to B.Cu
- moved R13 116.6 mm to (224.0, 127.5), turned to 180 degrees
- moved U13 113.4 mm to (10.5, 118.0)
- moved U14 113.4 mm to (-3.50, 124.0)
- moved U15 113.4 mm to (-3.50, 118.0)
- moved U16 113.4 mm to (-3.50, 112.0)
- moved U3 113.4 mm to (58.0, 118.0)
- moved U4 113.4 mm to (72.5, 112.0)
- moved U5 113.4 mm to (72.5, 118.0)
- moved U6 113.4 mm to (72.5, 124.0)
- moved U11 106.8 mm to (222.0, 137.5), turned to 90 degrees
- moved M1 105.5 mm to (358.5, 185.5)
- moved J1 100.2 mm to (113.5, 89.0)
- moved R8 95.5 mm to (254.0, 181.0), turned to 180 degrees
- moved R6 95.4 mm to (254.0, 173.0), turned to 180 degrees
- moved J3 94.0 mm to (246.5, 177.0)
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Connections:
- J11 pad 101: /KL46Z_DUAL/B18 -> (no net)
- J11 pad 102: /KL46Z_DUAL/A1 -> (no net)
- J11 pad 103: /KL46Z_DUAL/B19 -> (no net)
- J11 pad 104: /KL46Z_DUAL/A2 -> (no net)
- J11 pad 105: /KL46Z_DUAL/C0 -> (no net)
- J11 pad 107: /KL46Z_DUAL/C4 -> (no net)
- J11 pad 108: /KL46Z_DUAL/A12 -> (no net)
- J11 pad 109: /KL46Z_DUAL/C6 -> (no net)
- J11 pad 110: /KL46Z_DUAL/A4 -> (no net)
- J11 pad 111: /KL46Z_DUAL/C7 -> (no net)
- J11 pad 112: /KL46Z_DUAL/A5 -> (no net)
- J11 pad 113: /KL46Z_DUAL/C10 -> (no net)
- J11 pad 114: /KL46Z_DUAL/C8 -> (no net)
- J11 pad 115: /KL46Z_DUAL/C11 -> (no net)
- J11 pad 116: /KL46Z_DUAL/C9 -> (no net)
- J11 pad 201: /KL46Z_DUAL/C13 -> (no net)
- J11 pad 202: /KL46Z_DUAL/A13 -> (no net)
- J11 pad 203: /KL46Z_DUAL/C16 -> (no net)
- J11 pad 205: /KL46Z_DUAL/A7 -> (no net)
- J11 pad 207: /KL46Z_DUAL/A6 -> (no net)
- J11 pad 209: /KL46Z_DUAL/A14 -> (no net)
- J11 pad 211: /KL46Z_DUAL/A15 -> (no net)
- J11 pad 213: /KL46Z_DUAL/A16 -> (no net)
- J11 pad 215: /KL46Z_DUAL/A17 -> (no net)
- J11 pad 216: /KL46Z_DUAL/AREF -> (no net)
- J11 pad 217: /KL46Z_DUAL/B9 -> (no net)
- J11 pad 301: /KL46Z_DUAL/E31 -> (no net)
- J11 pad 302: /KL46Z_DUAL/SDA -> (no net)
- J11 pad 306: /KL46Z_DUAL/RST_b -> (no net)
- J11 pad 310: /KL46Z_DUAL/5V -> (no net)
- J11 pad 311: /KL46Z_DUAL/E6 -> (no net)
- J11 pad 405: /KL46Z_DUAL/E22 -> (no net)
- J11 pad 407: /KL46Z_DUAL/E23 -> (no net)
- J11 pad 409: /KL46Z_DUAL/B20 -> (no net)
- J11 pad 410: /KL46Z_DUAL/C2 -> (no net)
- J11 pad 412: /KL46Z_DUAL/C1 -> (no net)
Other:
- board size 200 x 160 mm -> 160 x 190 mm

Commit message: pcb seems about done.
Parts:
- moved U13 204.9 mm to (214.0, 142.0)
- moved U14 203.9 mm to (199.0, 148.0)
- moved U15 203.9 mm to (199.0, 142.0)
- moved U16 203.9 mm to (199.0, 136.0)
- moved M1 172.4 mm to (208.0, 101.5)
- moved U4 150.8 mm to (216.0, 158.5)
- moved U5 150.8 mm to (216.0, 164.5)
- moved U6 150.8 mm to (216.0, 170.5)
- moved U3 150.2 mm to (201.0, 164.0)
- moved D6 87.7 mm to (248.0, 73.0)
- moved J9 87.7 mm to (252.0, 75.0)
- moved L7 87.7 mm to (244.0, 79.0)
- moved D4 67.7 mm to (204.0, 73.0)
- moved J7 67.7 mm to (208.0, 75.0)
- moved L5 67.7 mm to (200.0, 78.0)
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
Commit message: pcb routing. choo choo. chugging along.
Parts:
- moved L6 17.3 mm to (172.0, 221.0)
- moved L3 16.5 mm to (172.0, 79.0)
- moved D5 10.3 mm to (168.0, 227.0), turned to 270 degrees
- moved J11 9.01 mm to (208.0, 167.0)
- moved L1 8.54 mm to (150.0, 93.5)
- moved D2 8.00 mm to (168.0, 73.0), turned to 270 degrees
- moved D1 6.50 mm to (204.0, 227.0)
- moved D3 6.50 mm to (248.0, 227.0)
- moved L2 6.50 mm to (200.0, 222.0)
- moved L4 6.50 mm to (244.0, 221.0)
- moved L8 3.00 mm to (150.0, 206.5), turned to 135 degrees
- moved L10 1.50 mm to (259.5, 206.5), turned to 65 degrees
- moved L9 1.50 mm to (259.5, 93.5), turned to 295 degrees
Routing:
- net +8V: track 0.00 -> 304.2 mm, vias 0 -> 2
- net N-00000149: track 0.00 -> 60.7 mm, vias 0 -> 2
- net N-00000166: track 0.00 -> 50.5 mm, vias 0 -> 1
- net N-00000186: track 0.00 -> 50.4 mm, vias 0 -> 1
- net N-00000164: track 0.00 -> 48.6 mm, vias 0 -> 4
- net N-00000151: track 0.00 -> 44.6 mm, vias 0 -> 4
- net N-0000050: track 0.00 -> 43.5 mm
- net N-00000136: track 0.00 -> 43.5 mm
- net N-00000160: track 0.00 -> 41.4 mm, vias 0 -> 4
- net N-00000158: track 0.00 -> 33.7 mm, vias 0 -> 4
- net N-00000150: track 0.00 -> 30.1 mm
- net N-00000157: track 0.00 -> 27.7 mm, vias 0 -> 2
- net N-00000159: track 0.00 -> 22.9 mm, vias 0 -> 2
- net N-00000161: track 0.00 -> 21.0 mm, vias 0 -> 2
- net N-00000165: track 0.00 -> 15.8 mm, vias 0 -> 1
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Other:
- rule trace_min: 0.254 -> 0.1

Commit message: shoot me plz. so many traces...
Routing:
- net /KL46Z_DUAL/M2_STEP: track 0.00 -> 139.0 mm, vias 0 -> 2
- net N-0000070: track 0.00 -> 111.8 mm, vias 0 -> 3
- net N-0000051: track 0.00 -> 111.1 mm, vias 0 -> 5
- net N-0000054: track 0.00 -> 110.7 mm, vias 0 -> 5
- net /KL46Z_DUAL/M3_STEP: track 0.00 -> 95.6 mm, vias 0 -> 3
- net /MOTOR3/FR: track 0.00 -> 84.4 mm, vias 0 -> 2
- net N-00000184: track 0.00 -> 71.0 mm, vias 0 -> 5
- net N-0000048: track 0.00 -> 70.1 mm, vias 0 -> 3
- net N-00000180: track 0.00 -> 61.6 mm, vias 0 -> 5
- net N-0000047: track 0.00 -> 59.5 mm, vias 0 -> 5
- net N-00000176: track 0.00 -> 52.1 mm, vias 0 -> 5
- net N-0000040: track 0.00 -> 48.0 mm, vias 0 -> 5
- net N-00000171: track 0.00 -> 43.9 mm, vias 0 -> 4
- net N-0000034: track 0.00 -> 43.7 mm, vias 0 -> 4
- net N-0000041: track 0.00 -> 37.0 mm
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
Commit message: All aboard the choo choo shoe.
Parts:
- moved J14 10.5 mm to (268.0, 156.0)
- moved J1 10.0 mm to (148.0, 144.0)
- moved J12 10.0 mm to (148.0, 156.0)
- moved J13 10.0 mm to (268.0, 144.0)
- moved C2 6.00 mm to (161.5, 112.5)
- moved C4 6.00 mm to (161.5, 173.5)
- moved C6 6.00 mm to (254.5, 126.5)
- moved C8 6.00 mm to (254.5, 187.5)
- moved R1 6.00 mm to (164.0, 133.5)
- moved R10 6.00 mm to (164.0, 167.0)
- moved R11 6.00 mm to (252.0, 105.5)
- moved R12 6.00 mm to (252.0, 133.0)
- moved R13 6.00 mm to (252.0, 166.5)
- moved R14 6.00 mm to (252.0, 194.0)
- moved R2 6.00 mm to (164.0, 106.0)
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Routing:
- net +8V: track 305.2 -> 17.0 mm, vias 4 -> 0
- net /KL46Z_DUAL/M2_STEP: track 139.0 -> 0.00 mm, vias 2 -> 0
- net /MOTOR2/SDIN: track 0.00 -> 136.3 mm, vias 0 -> 2
- net N-0000070: track 111.8 -> 1.27 mm, vias 3 -> 0
- net N-0000051: track 111.1 -> 1.27 mm, vias 5 -> 0
- net N-0000054: track 110.7 -> 1.27 mm, vias 5 -> 0
- net /KL46Z_DUAL/SDATA: track 0.00 -> 104.7 mm, vias 0 -> 2
- net /KL46Z_DUAL/SCL: track 0.00 -> 99.2 mm, vias 0 -> 9
- net /KL46Z_DUAL/M3_STEP: track 95.6 -> 0.00 mm, vias 3 -> 0
- net /XBEE0/RX: track 0.00 -> 86.7 mm, vias 0 -> 1
- net /XBEE0/TX: track 0.00 -> 85.2 mm
- net /MOTOR3/FR: track 84.4 -> 0.00 mm, vias 2 -> 0
- net /MOTOR0/CS: track 0.00 -> 83.3 mm, vias 0 -> 10
- net /MOTOR3/SDIN: track 0.00 -> 73.6 mm, vias 0 -> 2
- net /XBEE0/RESET_b: track 0.00 -> 67.8 mm, vias 0 -> 2
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
Commit message: pcb might be done.
Parts:
- added m3: , __m3, F.Cu at (135.0, 62.0)
- added m3: , __m3, F.Cu at (281.0, 62.0)
- added m3: , __m3, F.Cu at (135.0, 238.0)
- added m3: , __m3, F.Cu at (281.0, 238.0)
- added m3: , __m3, F.Cu at (203.8, 114.0)
- added m3: , __m3, F.Cu at (207.6, 188.7)
- moved R10 9.22 mm to (155.9, 162.6)
- moved C6 8.66 mm to (259.6, 133.5)
- moved C4 8.65 mm to (155.8, 167.0)
- moved R12 8.63 mm to (259.3, 137.6)
- moved C2 2.82 mm to (161.8, 109.7)
Routing:
- net +3.3V: track 0.00 -> 336.8 mm, vias 0 -> 17
- net /KL46Z_DUAL/M_VREF: track 0.00 -> 287.2 mm, vias 0 -> 15
- net /KL46Z_DUAL/M_OE_b: track 46.6 -> 331.7 mm, vias 4 -> 13
- net /KL46Z_DUAL/M_SRCLR_b: track 26.6 -> 233.5 mm, vias 3 -> 10
- net +8V: track 17.0 -> 204.0 mm, vias 0 -> 1
- net /KL46Z_DUAL/SCL: track 99.2 -> 247.2 mm, vias 9 -> 16
- net /KL46Z_DUAL/M2_STEP: track 0.00 -> 146.5 mm, vias 0 -> 2
- net N-0000069: track 0.00 -> 142.8 mm, vias 0 -> 5
- net /MOTOR0/CS: track 83.3 -> 223.4 mm, vias 10 -> 19
- net N-00000187: track 0.00 -> 129.4 mm, vias 0 -> 5
- net N-00000188: track 0.00 -> 128.1 mm, vias 0 -> 5
- net N-00000205: track 0.00 -> 127.3 mm, vias 0 -> 1
- net N-0000052: track 0.00 -> 124.8 mm, vias 0 -> 9
- net N-0000053: track 0.00 -> 119.3 mm, vias 0 -> 9
- net N-00000190: track 0.00 -> 117.1 mm, vias 0 -> 1
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- added copper zone on B.Cu, net GND

Commit message: 
Other:
- net class Default: via_drill 0.635 -> 0.5
- rule via_min_drill: 0.508 -> 0.5
Changed lines of the file:
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@@
     (links 244)
     (no_connects 5)
-    (area -0.100001 54.949999 500.100001 245.050001)
+    (area 127.949999 54.949999 288.050001 245.050001)
     (thickness 1.6)
-    (drawings 5)
+    (drawings 4)
     (tracks 1513)
     (zones 0)
@@
   )
   (setup
-    (last_trace_width 0.2)
+    (last_trace_width 0.254)
     (user_trace_width 0.1)
     (user_trace_width 0.2)
@@
     (edge_width 0.1)
     (via_size 0.889)
-    (via_drill 0.635)
+    (via_drill 0.5)
     (via_min_size 0.889)
-    (via_min_drill 0.508)
+    (via_min_drill 0.5)
     (uvia_size 0.508)
     (uvia_drill 0.127)
@@
     (visible_elements 7FFFFFFF)
     (pcbplotparams
-      (layerselection 3178497)
+      (layerselection 14712833)
       (usegerberextensions true)
       (excludeedgelayer true)
@@
       (outputformat 1)
       (mirror false)
-      (drillshape 1)
+      (drillshape 0)
       (scaleselection 1)
-      (outputdirectory "../../../../SYNC/Google Drive/ASU/kicad_svg/"))
+      (outputdirectory "C:/Users/Sev/Desktop/New folder (2)/"))
   )
   (net 0 "")
@@
     (trace_width 0.254)
     (via_dia 0.889)
-    (via_drill 0.635)
+    (via_drill 0.5)
     (uvia_dia 0.508)
     (uvia_drill 0.127)
@@
     )
   )
-  (gr_line (start 0 150) (end 500 150) (angle 90) (layer F.SilkS) (width 0.2))
   (gr_line (start 128 245) (end 128 55) (angle 90) (layer Edge.Cuts) (width 0.1))
   (gr_line (start 288 245) (end 128 245) (angle 90) (layer Edge.Cuts) (width 0.1))
